File: KiCad/ctLab.kicad_sch (KiCad schematic)
At the start: 0 parts

Commit message: kicad: add ctLab schematic parts
Parts:
- added C1, C14, C19, C2, C22, C23, C24, C3, C4, C5, C6, C7, C8: 100n ker. RMS, symbol Device:C
- added C10, C11, C12, C9: 470µ 35V, symbol Device:C_Polarized
- added C13, C15: 47µ 6V3, symbol Device:C_Polarized
- added C16, C17, C18, C21: 11µ 50V, symbol Device:C_Polarized
- added C20: 4µ7 35V, symbol Device:C_Polarized
- added D1, D3, D4: 1N4148, symbol Diode:1N4148
- added D2: 1N4004, symbol Diode:1N4004
- added JP1, JP2, JP3: Jumper, symbol Jumper:Jumper_2_Open
- added L1: 10µH axial, symbol Device:L
- added PL1: Pfosten 14-pol., symbol Connector_Generic:Conn_02x07_Odd_Even
- added PL2: Pfosten 10-pol., symbol Connector_Generic:Conn_02x05_Odd_Even
- added PL3: Schraubklemme RM 7,5, symbol Connector:Screw_Terminal_01x02
- added PL4: USB-B Printbuchse, symbol Connector:USB_B
- added R1: 0R (nur zum Test bestücken), symbol Device:R
- added R2, R3: 220R, symbol Device:R
- added R4: 2k7, symbol Device:R
- added R5: 2k2, symbol Device:R
- added R7: 4k7, symbol Device:R
- added R8: 10k, symbol Device:R
- added RB1, RB2, RB3: B80C1500, symbol Diode_Bridge:B80C1500G
- added RS1: D-Sub 9-pol. F, symbol Connector:DE9_Socket
- added TR1: Flachtrafo 2 x 15 V, 6 VA (Block), symbol Device:Transformer_1P_2S
- added TR2: Flachtrafo 2 x 9 V, 6 VA (Block), symbol Device:Transformer_1P_2S
- added U1: 7815, symbol Regulator_Linear:L7815
- added U10: XPort-01, symbol Connector_Generic:Conn_02x12_Odd_Even
- added U2: 7915, symbol Regulator_Linear:L7915
- added U3, U4: 7805, symbol Regulator_Linear:L7805
- added U5: FT232RL, symbol Interface_USB:FT232RL
- added U6: 6N137, symbol Isolator:6N137
- added U8: LF33, symbol Regulator_Linear:LF33_TO220
- added U9: MAX232, symbol Interface_UART:MAX232
