File: KiCad/ada-io.kicad_sch (KiCad schematic)
At the start: 36 parts, among them U12 ATmega32L-8P, U2 6N{136..137}

Commit message: cont. dcg schematic
Parts:
- U2: value 6N{136..137} -> ATmega32-16M; footprint (none) -> Package_DFN_QFN:QFN-44-1EP_7x7mm_P0.5mm_EP5.2x5.2mm
Connections:
- net DGnd: no longer U2.5 (GND)
- net DVcc: no longer U2.8 (VCC)
- net PD0: no longer U2.6 (VO)
- net at R2.2: no longer U2.3 (C)
- net at PL3.3 (Pin_3), PL3.4 (Pin_4): no longer U2.2 (A)
- new net: U2.17 (VCC), U2.38 (VCC), U2.5 (VCC)
- new net: U2.18 (GND), U2.39 (GND), U2.45 (GND), U2.6 (GND)
Changed lines of the file:
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@@
 		(dnp no)
 		(property "Reference" "U2"
-			(at 70.866 119.38 0)
+			(at 90.424 194.564 0)
 			(show_name no)
 			(do_not_autoplace no)
@@
 					(size 1.27 1.27)
 				)
+				(justify left)
 			)
 		)
-		(property "Value" "6N{136..137}"
-			(at 75.946 121.92 0)
+		(property "Value" "ATmega32-16M"
+			(at 90.424 196.596 0)
 			(show_name no)
 			(do_not_autoplace no)
@@
 					(size 1.27 1.27)
 				)
+				(justify left)
 			)
 		)
-		(property "Footprint" ""
+		(property "Footprint" "Package_DFN_QFN:QFN-44-1EP_7x7mm_P0.5mm_EP5.2x5.2mm"
+			(at 80.01 144.78 0)
+			(hide yes)
+			(show_name no)
+			(do_not_autoplace no)
+			(effects
+				(font
+					(size 1.27 1.27)
+					(italic yes)
+				)
+			)
+		)
+		(property "Datasheet" "http://ww1.microchip.com/downloads/en/DeviceDoc/doc2503.pdf"
 			(at 80.01 144.78 0)
 			(hide yes)
@@
 			)
 		)
-		(property "Datasheet" "https://www.vishay.com/docs/84732/6n137.pdf?utm_source=chatgpt.com"
+		(property "Description" "16MHz, 32kB Flash, 2kB SRAM, 1kB EEPROM, JTAG, QFN-44"
 			(at 80.01 144.78 0)
 			(hide yes)
-			(show_name no)
-			(do_not_autoplace no)
-			(effects
-				(font
-					(size 1.27 1.27)
-				)
-			)
-		)
-		(property "Description" "High Speed Optocoupler"
-			(at 81.28 124.46 0)
 			(show_name no)
 			(do_not_autoplace no)
@@
 		(pin "7"
 		)
+		(pin "16"
+		)
+		(pin "18"
+		)
+		(pin "27"
+		)
+		(pin "13"
+		)
+		(pin "14"
+		)
+		(pin "32"
+		)
+		(pin "22"
+		)
+		(pin "29"
+		)
+		(pin "11"
+		)
+		(pin "17"
+		)
+		(pin "9"
+		)
+		(pin "15"
+		)
+		(pin "21"
+		)
+		(pin "23"
+		)
+		(pin "10"
+		)
+		(pin "24"
+		)
+		(pin "25"
+		)
+		(pin "12"
+		)
+		(pin "19"
+		)
+		(pin "20"
+		)
+		(pin "26"
+		)
+		(pin "28"
+		)
+		(pin "30"
+		)
+		(pin "31"
+		)
+		(pin "33"
+		)
+		(pin "34"
+		)
+		(pin "35"
+		)
+		(pin "45"
+		)
+		(pin "42"
+		)
+		(pin "39"
+		)
+		(pin "38"
+		)
+		(pin "44"
+		)
+		(pin "37"
+		)
+		(pin "36"
+		)
+		(pin "40"
+		)
+		(pin "43"
+		)
+		(pin "41"
+		)
 		(instances

Commit message: Prefix KiCad component references
Parts:
- renumbered C2 to ADAIO.C2, C20 to ADAIO.C20, C25 to ADAIO.C25, C26 to ADAIO.C26, C27 to ADAIO.C27, C6 to ADAIO.C6, C7 to ADAIO.C7, CONN1 to ADAIO.CONN1, CONN2 to ADAIO.CONN2, CONN3 to ADAIO.CONN3, CONN4 to ADAIO.CONN4, CONN5 to ADAIO.CONN5, JP1 to ADAIO.JP1, JP2 to ADAIO.JP2, JP3 to ADAIO.JP3, JP4 to ADAIO.JP4, JP5 to ADAIO.JP5, L2 to ADAIO.L2, LED1 to ADAIO.LED1, PL1 to ADAIO.PL1, PL2 to ADAIO.PL2, PL3 to ADAIO.PL3, PL4 to ADAIO.PL4, PL5 to ADAIO.PL5, PL6 to ADAIO.PL6, R1 to ADAIO.R1, R2 to ADAIO.R2, R3 to ADAIO.R3, R4 to ADAIO.R4, R5 to ADAIO.R5, R6 to ADAIO.R6, R8 to ADAIO.R8, R9 to ADAIO.R9, U12 to ADAIO.U12, U2 to ADAIO.U2, XTAL1 to ADAIO.XTAL1
