File: KiCad/dcg.kicad_sch (KiCad schematic)
At the start: 8 parts, among them U10 LF411, U11 OP07, U13 CNY17-2, U2 ATmega32-16M, U3 LTC1864, U4 LT1019xN8, U5 NE5532, U7 6N137

Commit message: starting DCG
Parts:
- removed U10: LF411, Package_SO:SOIC-8_3.9x4.9mm_P1.27mm, symbol Amplifier_Operational:AD8015
- added C1, C11, C14, C15, C17, C18, C25, C28, C31, C4, C5, C8: 100n, symbol Device:C
- added C10: 4μ7 50V, symbol Device:C_Polarized
- added C13, C20: 100n 63V, symbol Device:C
- added C19, C22: 4µ7 25V Ta, symbol Device:C_Polarized
- added C2, C3: 22p, symbol Device:C
- added C23, C29: 100µ 63V, symbol Device:C_Polarized
- added C24: 220p, symbol Device:C
- added C27: 470p, symbol Device:C
- added C29: 2n2, symbol Device:C
- added C30: 330n, symbol Device:C
- added C30, C32, C33: 10µ 35V, symbol Device:C_Polarized
- added C6, C7: 220n, Capacitor_SMD:C_1206_3216Metric_Pad1.33x1.80mm_HandSolder, symbol Device:C
- added C9: 2n2, Capacitor_SMD:C_0805_2012Metric_Pad1.18x1.45mm_HandSolder, symbol Device:C
- added D1, D2, D3, D4: 1N4148, Diode_THT:D_DO-35_SOD27_P7.62mm_Horizontal, symbol Diode:1N4148
- added D10, LED1, LED2: LED, LED_THT:LED_D3.0mm, symbol Device:LED
- added D5, D6: 1N4007, Diode_THT:D_DO-41_SOD81_P10.16mm_Horizontal, symbol Diode:1N4007
- added D7: 1N5407, Diode_THT:D_DO-201AD_P15.24mm_Horizontal, symbol Diode:1N5407
- added JP1, JP2, JP3, JP4, JP5: Jumper_2_Open, symbol Jumper:Jumper_2_Open
- added L1: 16µH, symbol Device:L_Small
- added PL1: Conn_02x07_Odd_Even, symbol Connector_Generic:Conn_02x07_Odd_Even
- added PL2, PL3, PL4, PL5: Conn_02x05_Odd_Even, symbol Connector_Generic:Conn_02x05_Odd_Even
- added PL6: Conn_02x04_Top_Bottom, symbol Connector_Generic:Conn_02x04_Top_Bottom
- added PL7: Screw_Terminal_01x04, symbol Connector:Screw_Terminal_01x04
- added Q1, Q10, Q11, Q2: BS170, Package_TO_SOT_THT:TO-92_Inline, symbol Transistor_FET:BS170
- added Q12: BD243B, BD243C, Package_TO_SOT_THT:TO-220-3_Horizontal_TabDown, symbol Transistor_BJT:BD249
- added Q3, Q4, Q7: BC546, Package_TO_SOT_THT:TO-92_Inline, symbol Transistor_BJT:BC546
- added Q5: BC556, Package_TO_SOT_THT:TO-92_Inline, symbol Transistor_BJT:BC556
- added Q6: BD677, Package_TO_SOT_THT:TO-220-3_Horizontal_TabDown, symbol Transistor_BJT:BC517
- added Q8, Q9: IRF540N, Package_TO_SOT_THT:TO-220-3_Vertical, symbol Transistor_FET:IRF540N
- added R10, R11, R12, R29, R52: 2k2, symbol Device:R
- added R10, R11, R13, R15: 470R, Resistor_SMD:R_0805_2012Metric, symbol Device:R
- added R12, R21, R22, R24: 30k, symbol Device:R
- added R14: 100k, Resistor_SMD:R_0805_2012Metric, symbol Device:R
- added R16: 7k5, symbol Device:R
- added R17: 20k, symbol Device:R
- added R18, R19, R20, R23, R26, R31, R37, R42, R43, R44, R47, R50, R61: 10k, symbol Device:R
- added R25, R32, R33, R40, R49: 1k, symbol Device:R
- added R27: 39k, symbol Device:R
- added R28, R36: 10k, symbol Device:R_Trim
- added R30: 12k, symbol Device:R
- added R34: 3k, symbol Device:R
- added R35: 6k8, symbol Device:R
- added R38, R6: 10R, symbol Device:R
- added R39: 330R, symbol Device:R
- added R41: 1k8, symbol Device:R
- added R45: 22k, symbol Device:R
- added R46, R48, R9: 4k7, symbol Device:R
- added R53: 4R7 2W, symbol Device:R
- added R54: 47R, symbol Device:R
- added R55, R8: 470R, symbol Device:R
- added R56, R57: 470m 5W, symbol Device:R
- added R58: 2R2, symbol Device:R
- added R59, R60: 100R, symbol Device:R
- added R62: 180k, symbol Device:R
- added R7: 0R, symbol Device:R
- added U10, U6: LF411, Package_DIP:DIP-8_W10.16mm, symbol ctLab:LF411
- added U12: DG409, DG509, symbol CERN:DG409
- added U14: LF412-N, symbol Amplifier_Operational:NE5532
- added U7: LTC1655, symbol Analog_DAC:LTC1257
- added U8: DG413, symbol CERN:DG413
- added XTAL2: 16MHz HC-49U, symbol CERN:Quartz Crystal
- added ZD1: ZPD 9V1 400mW, Diode_THT:D_DO-35_SOD27_P10.16mm_Horizontal, symbol Diode:ZPDxx
- renumbered U7 to U1
Connections:
- new net: C2.2, XTAL2.1 (OSC1)
- new net: C3.2, XTAL2.2 (OSC2)
- new net AGnd: PL1.7 (Pin_7), PL1.8 (Pin_8)
- new net DGnd: C2.1, C3.1, PL1.11 (Pin_11), PL1.12 (Pin_12), PL1.3 (Pin_3), PL1.4 (Pin_4)
- new net DVcc: PL1.13 (Pin_13), PL1.14 (Pin_14)
- new net DVgl+: PL1.1 (Pin_1), PL1.2 (Pin_2)
- new net V++: PL1.5 (Pin_5), PL1.6 (Pin_6)
- new net V--: PL1.10 (Pin_10), PL1.9 (Pin_9)
Other:
- moved on the sheet: U1, U11, U13, U2, U3, U4, U5A, U5B

Commit message: cont. dcg schematic
Parts:
- removed R28, R36: 10k, symbol Device:R_Trim
- added R24: 30k, symbol Device:R
- added R28, R36: 10k, symbol Device:R_Potentiometer_Trim
- added R45b, R45c, R45d: 22k, symbol Device:R
- added RV1: R_Potentiometer_Trim, symbol Device:R_Potentiometer_Trim
- added U15: LF411, Package_DIP:DIP-8_W10.16mm, symbol ctLab:LF411
- added U16, U9: LF412A, Package_DIP:DIP-8_W10.16mm, symbol ctLab:LF412A
- added unit 2 of U8
- added unit 4 of U8
- added unit 5 of U8
- added unit 3 of U8
- Q8, Q9: value IRF540N -> IRF540
- R55: renamed from R56; value 470m 5W -> 470R
- U3: footprint (none) -> Package_SO:SOIC-8_5.3x5.3mm_P1.27mm
- renumbered R45 to R45a
Connections:
- net AGnd: now also C20.1, C7.2, R33.2, R53.2, R54.2, R55.2, R57.2, U3.3 (IN^{-}), U3.4 (GND), U7.5 (GND), U8.5 (GND)
- net DGnd: now also JP1.1 (A), JP2.1 (A), JP3.1 (A)
- net S1A: now reaches R45a.1
- net S1A: now also Q8.1 (G), U12.4 (S1A)
- net MuxGnd: now reaches R45a.2
- net MuxGnd: now also C11.1, C22.2, Q1.3 (S), R12.2, U12.15 (GND), U2.28 (AGND), ZD1.2 (A), R45b.2, R45c.2, R45d.2
- net at Q1.1 (D): now also R16.2
- net MOSI: now reaches Q1.2 (G)
- net MOSI: now also U2.1 (PB5)
- net ICP: now reaches JP2.2 (B)
- net ICP: now also U2.15 (PD6)
- net at R15.1: now also R14.2, U3.2 (IN^{+})
- net at R15.2: now also U16.6 (In-), U16.7 (OUT)
- net ADC2: now reaches R16.1
- net ADC2: now also C11.2, R12.1, U2.35 (PA2), R24.2, U8.6 (S4)
- net S1B: now reaches R57.1
- net S1B: now also Q8.3 (S), U12.13 (S1B)
- net MPXU: now reaches U8.1 (IN)
- net MPXU: now also U2.23 (PC4)
- net at U8.2 (D): now also U7.7 (VOUT), U8.15 (D)
- net at U8.3 (S): now also R19.1
- net at R26.1: now also U8.14 (S)
- net at R26.2: now also C20.2, U9.3 (In+)
- net at R14.1: now also C7.1, U3.1 (V_{REF}), U7.6 (VREF)
- net at XTAL2.1 (OSC1): now also C3.2, U2.7 (XTAL2); no longer C2.2
- net at XTAL2.2 (OSC2): now also C2.2, U2.8 (XTAL1); no longer C3.2
- net at Q11.1 (D): now also Q10.1 (D), Q8.2 (D), Q9.2 (D)
- net S4A: now reaches Q11.2 (G)
- net S4A: now also U12.7 (S4A), R45d.1
- net S4B: now reaches Q11.3 (S)
- net S4B: now also R55.1, U12.10 (S4B)
- net MuxPwr: now reaches ZD1.1 (K)
- net MuxPwr: now also C22.1, R46.2, U12.14 (V+), U12.2 (EN), U12.8 (DA)
- net V+: now reaches R46.1
- net S3A: now reaches Q10.2 (G)
- net S3A: now also U12.6 (S3A), R45c.1
- net S3B: now reaches Q10.3 (S)
- net S3B: now also R54.1, U12.11 (S3B)
- net PB0: now reaches U7.1 (CKL)
- net PB0: now also R10.2, U2.40 (PB0)
- net PB1: now reaches U7.2 (DIN)
- net PB1: now also U2.41 (PB1)
- net PB4: now reaches U7.3 (~{LOAD})
- net PB4: now also U2.44 (PB4)
- net DVccDAC: now reaches U7.8 (VCC)
- net DVccDAC: now also U3.8 (V_{CC}), U8.12 (VL)
- net at R34.1: now also U9.1 (OUT), U9.2 (In-)
- net at R34.2: now also R33.1, U10.3 (In+)
- net at R11.1: now also U3.6 (SDO)
- net MISO: now reaches R11.2
- net MISO: now also U2.2 (PB6)
- net MPXA0: now reaches U12.1 (A0)
- net MPXA0: now also U2.21 (PC2)
- net S2B: now reaches U12.12 (S2B)
- net S2B: now also Q9.3 (S), R53.1
- net MPXA1: now reaches U12.16 (A1)
- net MPXA1: now also U2.22 (PC3)
- net V-: now reaches U12.3 (V-)
- net S2A: now reaches U12.5 (S2A)
- net S2A: now also Q9.1 (G), R45b.1
- net MPXDB: now reaches U12.9 (DB)
- net at U10.1 (N1): now also R28.1
- net at U10.4 (VCC-): now also R28.2
- net at U10.5 (N2): now also R28.3
- net at U10.6 (OUT): now also D4.1 (K)
- net at U3.5 (CONV): now also R13.1
- net at U3.7 (SCK): now also R10.1
- net PD1: now reaches U2.10 (PD1)
- net INT0: now reaches U2.11 (PD2)
- net INT1: now reaches U2.12 (PD3)
- net OC1B: now reaches U2.13 (PD4)
- net OC1A: now reaches U2.14 (PD5)
- net OC1A: now also JP1.2 (B)
- net OC2: now reaches U2.16 (PD7)
- net OC2: now also JP3.2 (B)
- net GND: now reaches U2.18 (GND), U2.39 (GND), U2.45 (GND), U2.6 (GND)
- net GND: no longer U2.28 (GND)
- net PC0: now reaches U2.19 (PC0)
- net PC1: now reaches U2.20 (PC1)
- net MPXI: now reaches U2.24 (PC5)
- net MPXI: now also U8.16 (IN)
- net MPX1864: now reaches U2.25 (PC6)
- net MPX1864: now also U8.8 (IN), U8.9 (IN)
- net OutputEnable: now reaches U2.26 (PC7)
- net ARef: now reaches U2.29 (AREF)
- net PB7: now reaches U2.3 (PB7)
- net PB7: now also R13.2
- net ADC7: now reaches U2.30 (PA7)
- net ADC6: now reaches U2.31 (PA6)
- net ADC5: now reaches U2.32 (PA5)
- net ADC4: now reaches U2.33 (PA4)
- net ADC3: now reaches U2.34 (PA3)
- net ADC3: now also U8.11 (S3)
- net ADC1: now reaches U2.36 (PA1)
- net ADC0: now reaches U2.37 (PA0)
- net RESET: now reaches U2.4 (~{RESET})
- net INT2: now reaches U2.42 (PB2)
- net OC0: now reaches U2.43 (PB3)
- net PD0: now reaches U2.9 (PD0)
- new net: U16.5 (In+), U8.10 (D3), U8.7 (D4)
- new net: U8.13 (V+), U9.8 (V+)
- new net: U8.4 (V-), U9.4 (V-)
- new net X3Out: R24.1
- no-connect marks 0 -> 4
Other:
- note added: "0..1.024 V"
- note added: "Analog/Digital Converter"
- note added: "Buffer"
- note added: "Current Control"
- note added: "Current Sense Amp"
- note added: "Digital/Analog Converter"
- note added: "MPX A/D Current"
- note added: "MPX A/D Voltage"
- note added: "Module Address"
- note added: "Offset"
- note added: "Reference Voltage"
- note added: "Voltage Control"
- note added: "Voltage Range Sw A/D"
- moved on the sheet: C11, C20, C22, C7, D4, PL7, Q1, Q10, Q11, Q8, Q9, R10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

Commit message: Prefix KiCad component references
Parts:
- removed C29: 2n2, symbol Device:C
- removed D2: 1N4148, Diode_THT:D_DO-35_SOD27_P7.62mm_Horizontal, symbol Diode:1N4148
- removed R52: 2k2, symbol Device:R
- removed U10, U6: LF411, Package_DIP:DIP-8_W10.16mm, symbol ctLab:LF411
- added DCG.C16: 10µ 35V, symbol Device:C_Polarized
- added DCG.C2: 2n2, Capacitor_SMD:C_0805_2012Metric_Pad1.18x1.45mm_HandSolder, symbol Device:C
- added DCG.D2: 1N4148, Diode_THT:D_DO-35_SOD27_P7.62mm_Horizontal, symbol Diode:1N4148
- added DCG.LED3: LED, LED_THT:LED_D3.0mm, symbol Device:LED
- added DCG.R51: 220R, symbol Device:R
- added DCG.R52: 2k2, symbol Device:R
- added DCG.R56: 0R47 5W, symbol Device:R
- added DCG.U10: LF411, Package_DIP:DIP-8_W10.16mm, symbol ctLab:LF411
- renumbered C1 to DCG.C1, C10 to DCG.C10, C11 to DCG.C11, C13 to DCG.C13, C14 to DCG.C14, C15 to DCG.C15, C17 to DCG.C17, C18 to DCG.C18, C19 to DCG.C19, C2 to DCG.C2, C20 to DCG.C20, C22 to DCG.C22, C23 to DCG.C23, C24 to DCG.C24, C25 to DCG.C25, C27 to DCG.C27, C28 to DCG.C28, C29 to DCG.C29, C3 to DCG.C3, C30 to DCG.C30, C31 to DCG.C31, C32 to DCG.C32, C33 to DCG.C33, C4 to DCG.C4, C5 to DCG.C5, C6 to DCG.C6, C7 to DCG.C7, C8 to DCG.C8, C9 to DCG.C9, D1 to DCG.D1, D10 to DCG.D10, D3 to DCG.D3, D4 to DCG.D4, D5 to DCG.D5, D6 to DCG.D6, D7 to DCG.D7, JP1 to DCG.JP1, JP2 to DCG.JP2, JP3 to DCG.JP3, JP4 to DCG.JP4, JP5 to DCG.JP5, L1 to DCG.L1, LED1 to DCG.LED1, LED2 to DCG.LED2, PL1 to DCG.PL1, PL2 to DCG.PL2, PL3 to DCG.PL3, PL4 to DCG.PL4, PL5 to DCG.PL5, PL6 to DCG.PL6, PL7 to DCG.PL7, Q1 to DCG.Q1, Q10 to DCG.Q10, Q11 to DCG.Q11, Q12 to DCG.Q12, Q2 to DCG.Q2, Q3 to DCG.Q3, Q4 to DCG.Q4, Q5 to DCG.Q5, Q6 to DCG.Q6, Q7 to DCG.Q7, Q8 to DCG.Q8, Q9 to DCG.Q9, R10 to DCG.R10, R11 to DCG.R11, R12 to DCG.R12, R13 to DCG.R13, R14 to DCG.R14, R15 to DCG.R15, R16 to DCG.R16, R17 to DCG.R17, R18 to DCG.R18, R19 to DCG.R19, R20 to DCG.R20, R21 to DCG.R21, R22 to DCG.R22, R23 to DCG.R23, R24 to DCG.R24, R25 to DCG.R25, R26 to DCG.R26, R27 to DCG.R27, R28 to DCG.R28, R29 to DCG.R29, R30 to DCG.R30, R31 to DCG.R31, R32 to DCG.R32, R33 to DCG.R33, R34 to DCG.R34, R35 to DCG.R35, R36 to DCG.R36, R37 to DCG.R37, R38 to DCG.R38, R39 to DCG.R39, R40 to DCG.R40, R41 to DCG.R41, R42 to DCG.R42, R43 to DCG.R43, R44 to DCG.R44, R45a to DCG.R45a, R45b to DCG.R45b, R45c to DCG.R45c, R45d to DCG.R45d, R46 to DCG.R46, R47 to DCG.R47, R48 to DCG.R48, R49 to DCG.R49, R50 to DCG.R50, R53 to DCG.R53, R54 to DCG.R54, R55 to DCG.R55, R57 to DCG.R57, R58 to DCG.R58, R59 to DCG.R59, R6 to DCG.R6, R60 to DCG.R60, R61 to DCG.R61, R62 to DCG.R62, R7 to DCG.R7, R8 to DCG.R8, R9 to DCG.R9, RV1 to DCG.RV1, U1 to DCG.U1, U11 to DCG.U11, U12 to DCG.U12, U13 to DCG.U13, U14 to DCG.U14, U15 to DCG.U15, U16 to DCG.U16, U2 to DCG.U2, U3 to DCG.U3, U4 to DCG.U4, U5 to DCG.U5, U7 to DCG.U7, U8 to DCG.U8, U9 to DCG.U9, XTAL2 to DCG.XTAL2, ZD1 to DCG.ZD1
Connections:
- net ADC3: now also DCG.C8.2, DCG.R44.2
- net AGnd: now also DCG.C23.2, DCG.C28.1, DCG.C29.2, DCG.C8.1, DCG.D5.1 (K), DCG.PL6.4 (Pin_4), DCG.Q3.3 (E), DCG.R20.2, DCG.R48.2, DCG.R50.1, DCG.C16.2
- net INT2: now also DCG.PL6.7 (Pin_7)
- net MPXDB: now also DCG.R41.2, DCG.R43.1
- net OC0: now also DCG.PL6.8 (Pin_8)
- net PC0: now also DCG.PL6.5 (Pin_5)
- net PC1: now also DCG.PL6.6 (Pin_6)
- net V+: now also DCG.U11.7 (V+), DCG.U10.7 (VCC+)
- net V++: now also DCG.D3.2 (A), DCG.R38.2, DCG.C16.1
- net V-: now also DCG.U11.4 (V-)
- net PwrIn+: now reaches DCG.C29.1
- net PwrIn+: now also DCG.C27.2, DCG.C28.2, DCG.PL6.1 (Pin_1), DCG.Q6.2 (C), DCG.D2.2 (A)
- net ConstantPwr+: now reaches DCG.C23.1
- net ConstantPwr+: now also DCG.D3.1 (K), DCG.R37.1, DCG.R39.1, DCG.D2.1 (K), DCG.LED3.2 (A)
- net at DCG.R41.1: now also DCG.R40.2, DCG.U10.2 (In-)
- net at DCG.R39.2: now also DCG.Q5.3 (E)
- net at DCG.R42.1: now also DCG.R50.2, DCG.U11.2 (-)
- net at DCG.R42.2: now also DCG.R44.1, DCG.U11.6
- net PwrBasis: now reaches DCG.PL6.2 (Pin_2)
- net PwrBasis: now also DCG.Q6.1 (E), DCG.R51.1
- net PwrEmitter: now reaches DCG.PL6.3 (Pin_3)
- net PwrEmitter: now also DCG.R52.2, DCG.R56.1
- net at DCG.U13.1: now also DCG.LED2.2 (A), DCG.R32.1
- net at DCG.U13.2: now also DCG.D4.2 (A)
- net Out-: now reaches DCG.Q10.1 (D), DCG.Q11.1 (D), DCG.Q8.2 (D), DCG.Q9.2 (D)
- net Out-: now also DCG.C30.2, DCG.D6.2 (A), DCG.D7.2 (A), DCG.PL7.4 (Pin_4)
- net at DCG.D1.1 (K): now also DCG.R25.2
- net at DCG.D1.2 (A): now also DCG.LED2.1 (K)
- net Out+: now reaches DCG.PL7.1 (Pin_1)
- net Out+: now also DCG.D7.1 (K), DCG.R49.2, DCG.R51.2, DCG.R56.2
- net Sense+: now reaches DCG.PL7.2 (Pin_2)
- net Sense-: now reaches DCG.PL7.3 (Pin_3)
- net at DCG.C27.1: now also DCG.Q5.1 (C), DCG.Q6.3 (B), DCG.Q7.1 (C)
- net at DCG.R49.1: now also DCG.Q7.2 (B), DCG.R52.1
- net at DCG.R37.2: now also DCG.Q5.2 (B), DCG.LED3.1 (K)
- net at DCG.D6.1 (K): now also DCG.D5.2 (A)
- net at DCG.R33.1, DCG.R34.2: now also DCG.U10.3 (In+)
- net at DCG.U11.3 (+): now also DCG.R43.2
- net at DCG.R40.1: now also DCG.C24.1
- net at DCG.R28.1: now also DCG.U10.1 (B1)
- net at DCG.R28.2: now also DCG.U10.4 (VCC-)
- net at DCG.R28.3: now also DCG.U10.5 (B2)
- net at DCG.D4.1 (K): now also DCG.C24.2, DCG.U10.6 (OUT)
- net at DCG.R25.1: now also DCG.C2.2
- no-connect marks 4 -> 6
Other:
- note added: "Current Source"
- note added: "X2 Current A/D Amp"
- moved on the sheet: DCG.C23, DCG.C24, DCG.C27, DCG.C28, DCG.C29, DCG.C30, DCG.C8, DCG.D1, DCG.D3, DCG.D4, DCG.D5, DCG.D6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

Commit message: cont. drafting DCG schematic
Parts:
- added DCG.C21, DCG.C26: 10μ 35V, symbol Device:C_Polarized
- added DCG.PL1: Conn_02x07_Odd_Even, symbol Connector_Generic:Conn_02x07_Odd_Even
- added DCG.R1, DCG.R3: 2k2, symbol Device:R
- added DCG.R45: 10k, symbol Device:R_Potentiometer_Trim
- added DCG.U6: LF411, Package_DIP:DIP-8_W10.16mm, symbol ctLab:LF411
- DCG.U4: value LT1019xN8 -> LT1019xN8 or ADREF43
- renumbered DCG.C2 to DCG.C12
Connections:
- net RESET is gone; now on net ~{RESET}: DCG.U2.4 (~{RESET})
- net ADC0: now also DCG.PL4.1 (Pin_1)
- net ADC1: now also DCG.PL4.2 (Pin_2)
- net AGnd: now also DCG.C13.1, DCG.C15.1, DCG.C17.1, DCG.C18.1, DCG.C19.2, DCG.C25.1, DCG.R47.2, DCG.U13.4, DCG.U4.4 (GND), DCG.C21.1, DCG.C26.2
- net DGnd: now also DCG.PL4.7 (Pin_7), DCG.PL4.9 (Pin_9), DCG.PL5.10 (Pin_10), DCG.PL5.4 (Pin_4), DCG.PL5.6 (Pin_6), DCG.PL5.8 (Pin_8)
- net INT0: now also DCG.PL4.3 (Pin_3)
- net INT1: now also DCG.PL4.4 (Pin_4)
- net MISO: now also DCG.PL5.9 (Pin_9)
- net MOSI: now also DCG.PL5.1 (Pin_1)
- net OC1B: now also DCG.R47.1, DCG.U13.5
- net PB7: now also DCG.PL5.7 (Pin_7)
- net PC0: now also DCG.PL4.6 (Pin_6), DCG.R3.2
- net PC1: now also DCG.PL4.5 (Pin_5), DCG.R1.2
- net V--: now also DCG.R6.2
- net DCG.PL4:Vcc: now reaches DCG.PL5.2 (Pin_2)
- net DCG.PL4:Vcc: now also DCG.C1.2, DCG.C10.1, DCG.C14.2, DCG.C4.2, DCG.L1.2, DCG.PL4.10 (Pin_10), DCG.PL4.8 (Pin_8), DCG.R9.1, DCG.U2.17 (VCC), DCG.U2.38 (VCC), DCG.U2.5 (VCC), DCG.R1.1, DCG.R3.1
- net ~{RESET}: now reaches DCG.PL5.5 (Pin_5)
- net ~{RESET}: now also DCG.R9.2
- net DCG.PL1:DGnd: now reaches DCG.C4.1
- net DCG.PL1:DGnd: now also DCG.C1.1, DCG.C10.2, DCG.C14.1, DCG.R7.2, DCG.PL1.11 (Pin_11), DCG.PL1.12 (Pin_12), DCG.PL1.3 (Pin_3), DCG.PL1.4 (Pin_4)
- net at DCG.R6.1: now also DCG.C15.2, DCG.R28.2, DCG.C21.2, DCG.U6.4 (VCC-)
- net at DCG.R28.1: now also DCG.U6.5 (B2); no longer DCG.U10.1 (B1)
- net DCG.U10:3: now reaches DCG.R33.1, DCG.R34.2, DCG.U10.3 (In+)
- net at DCG.U10.4 (VCC-): now also DCG.R45.2; no longer DCG.R28.2
- net at DCG.R28.3: now also DCG.U6.1 (B1); no longer DCG.U10.5 (B2)
- net at DCG.C12.1: now also DCG.R17.1, DCG.U6.2 (In-)
- net DCG.U2a:27: now reaches DCG.U4.2 (IN)
- net DCG.U2a:27: now also DCG.C17.2, DCG.C19.1, DCG.C5.1, DCG.L1.1, DCG.U2.27 (AVCC)
- net DCG.U4:OUT: now reaches DCG.U4.6 (OUT)
- net DCG.PL1:AGnd: now reaches DCG.C5.2
- net DCG.PL1:AGnd: now also DCG.R7.1, DCG.PL1.7 (Pin_7), DCG.PL1.8 (Pin_8)
- net DCG.U13:1: now reaches DCG.LED2.2 (A), DCG.R32.1, DCG.U13.1
- net DCG.U13:1: now also DCG.R17.2, DCG.R23.1
- net DCG.D4:A: now reaches DCG.D4.2 (A), DCG.U13.2
- net DCG.R19:1: now reaches DCG.R19.1, DCG.U8.3 (S)
- net DCG.R26:1: now reaches DCG.R26.1, DCG.U8.14 (S)
- net at DCG.C25.2: now also DCG.C18.2, DCG.R38.1, DCG.C26.1, DCG.U6.7 (VCC+)
- net at DCG.D1.1 (K), DCG.R25.2: now also DCG.U6.6 (OUT)
- net at DCG.R19.2: now also DCG.C13.2, DCG.U6.3 (In+)
- new net: DCG.R45.3, DCG.U10.1 (B1)
- new net: DCG.R45.1, DCG.U10.5 (B2)
- new net DCG.PL1:DVcc: DCG.PL1.13 (Pin_13), DCG.PL1.14 (Pin_14)
- new net DCG.PL1:DVgl+: DCG.PL1.1 (Pin_1), DCG.PL1.2 (Pin_2)
- new net DCG.PL1:V++: DCG.PL1.5 (Pin_5), DCG.PL1.6 (Pin_6)
- new net DCG.PL1:V--: DCG.PL1.10 (Pin_10), DCG.PL1.9 (Pin_9)
- no-connect marks 6 -> 9
Other:
- note added: "2.5000V"
- note added: "Current Mode IF"
- note added: "Der Mikrocontroller ATmega 32 (U2) besorgt die Kommunikation mit dem c't-Lab-OptoBus, er versteht die schon vom ADA-IOund DDS-Modul bekannte c'tLab-Syntax und steuert die D/A-Wandler-Kanäle, Multiplexer und Umschalter, kümmert sich um Bedieneingaben am PM8-Panel und liest die Ist-Werte der A/DKanäle aus."
- note added: "Der im Regelkreis liegende Optokoppler U13 meldet die einsetzende Strombegrenzung an den Prozessor, der daraufhin die rote „I"- LED auf dem Bedienpanel anknipst und das „Overload"-Flag für die Statusmeldung setzt."
- note added: "Die Spannung am ausgewählten Shunt gelangt an OpAmp U10, der bei Überschreiten der vom D/A-Wandler vorgegebenen Spannung den Ausgang herunterregelt, bis der Sollstrom erreicht ist - realisiert durch eine Dioden-VerODERrung (D1, D4) am Level-Shifter Q4."
- note added: "U11 verstärkt die Shunt-Spannung um den Faktor zwei, am Istwert-A/D-Wandler kommen also knapp 2 V an, wenn ein Strom von 2 A durch R57 (0,47 Ohm) fließt."
- note added: "die Ausgangsspannung des D/A-Wandlers kann nicht stabiler sein als die ihm zugeführte Referenzspannung."
- moved on the sheet: DCG.C12, DCG.C2, DCG.C20, DCG.C24, DCG.C3, DCG.C30, DCG.C31, DCG.C32, DCG.C33, DCG.C6, DCG.C9, DCG.D1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

Commit message: finishing dcg schematic and repairing IFP schematic
Parts:
- removed DCG.C30, DCG.C32, DCG.C33: 10µ 35V, symbol Device:C_Polarized
- removed DCG.C31: 100n, symbol Device:C
- removed DCG.D10: LED, LED_THT:LED_D3.0mm, symbol Device:LED
- removed DCG.PL1: Conn_02x07_Odd_Even, symbol Connector_Generic:Conn_02x07_Odd_Even
- removed DCG.R10, DCG.R11, DCG.R12: 2k2, symbol Device:R
- removed DCG.R24: 30k, symbol Device:R
- removed DCG.R36: 10k, symbol Device:R_Potentiometer_Trim
- removed DCG.R55: 470R, symbol Device:R
- removed DCG.RV1: R_Potentiometer_Trim, symbol Device:R_Potentiometer_Trim
- removed DCG.U14: LF412-N, symbol Amplifier_Operational:NE5532
- removed DCG.U15: LF411, Package_DIP:DIP-8_W10.16mm, symbol ctLab:LF411
- added C31: 100n, symbol Device:C
- added DCG.R2, DCG.R4: 220R, symbol Device:R
- added R5: 2k7, symbol Device:R
- renumbered DCG.R45 to DCG.R36
Connections:
- net ADC4: now also DCG.R61.1, DCG.R62.2, C31.1
- net AGnd: now also DCG.C6.2, DCG.C9.2, DCG.Q2.3 (S), DCG.R29.2, DCG.R30.2
- net DCG.U13:1: now also DCG.U5.1
- net DGnd: now also DCG.U1.6 (VO)
- net DVcc: now also DCG.R8.1, DCG.U1.8 (VCC), R5.1
- net DVccDAC: now also DCG.C6.1
- net GND: now also DCG.R61.2, C31.2
- net INT0: now also DCG.LED1.1 (K)
- net MOSI: now also DCG.Q2.2 (G)
- net Out+: now also DCG.Q7.3 (E), DCG.R48.1, DCG.R58.1, DCG.R60.2
- net Out-: now also DCG.C30.1, DCG.R59.2; no longer DCG.Q11.1 (D), DCG.Q8.2 (D), DCG.Q9.2 (D)
- net OutputEnable: now also DCG.R29.1, DCG.R31.1
- net PD0: now also DCG.U1.7 (EN), R5.2
- net PD1: now also DCG.R4.2
- net PwrBasis: now also DCG.Q12.1 (B)
- net PwrEmitter: now also DCG.Q12.3 (E)
- net PwrIn+: now also DCG.Q12.2 (C), DCG.R62.1
- net Sense-: now also DCG.R59.1, DCG.U5.5 (+)
- net at DCG.C30.2: now also DCG.R58.2
- net at DCG.PL3.1 (Pin_1): now also DCG.PL3.2 (Pin_2), DCG.R2.1
- net at DCG.PL3.10 (Pin_10): now also DCG.JP5.1 (A), DCG.PL2.10 (Pin_10), DCG.PL2.9 (Pin_9), DCG.PL3.9 (Pin_9)
- net at DCG.PL3.3 (Pin_3): now also DCG.PL3.4 (Pin_4), DCG.U1.2 (A)
- net at DCG.PL3.7 (Pin_7): now also DCG.JP4.1 (A), DCG.PL2.7 (Pin_7), DCG.PL2.8 (Pin_8), DCG.PL3.8 (Pin_8)
- net at DCG.R20.1: now also DCG.R21.1, DCG.U5.3 (+)
- net at DCG.C12.1, DCG.R17.1, DCG.U6.2 (In-): now also DCG.R18.1
- net at DCG.R31.2: now also DCG.Q3.2 (B)
- net at DCG.R14.2, DCG.R15.1, DCG.U3.2 (IN^{+}): now also DCG.C9.1
- net at DCG.R27.1: now also DCG.Q4.2 (B), DCG.R30.1
- net DCG.Q6:B: now reaches DCG.R27.2
- net DCG.Q6:B: now also DCG.C27.1, DCG.Q4.1 (C), DCG.Q5.1 (C), DCG.Q6.3 (B), DCG.Q7.1 (C)
- net at DCG.R60.1: now also DCG.R21.2
- net at DCG.Q3.1 (C): now also DCG.R35.2
- net at DCG.U5.6 (-): now also DCG.R22.2, DCG.U5.7
- net at DCG.Q2.1 (D): now also DCG.R18.2
- net at DCG.R35.1: now also DCG.LED3.1 (K), DCG.Q5.2 (B), DCG.R37.2
- net at DCG.PL2.1 (Pin_1): now also DCG.JP4.2 (B), DCG.PL2.2 (Pin_2), DCG.R4.1
- net at DCG.PL2.3 (Pin_3): now also DCG.JP5.2 (B), DCG.PL2.4 (Pin_4)
- net at DCG.R8.2: now also DCG.LED1.2 (A)
- net at DCG.U1.3 (C): now also DCG.R2.2
- net at DCG.R23.2: now also DCG.R22.1, DCG.U5.2 (-)
- net at DCG.R32.2: now also DCG.Q4.3 (E)
- new net: DCG.Q11.1 (D), DCG.Q8.2 (D), DCG.Q9.2 (D)
- no-connect marks 9 -> 15
Other:
- note added: "Activity LED"
- note added: "Der D/A-Wandler LTC1655 wird doppelt genutzt: über einen Multiplexer mit nachfolgenden Sample&Hold-Stufen steuert er abwechselnd den Soll-Strom und die Sollspannung, die Ausgabe erfolgt im 1-ms-Interrupt des Controllers, nach zwei Millisekunden sind also beide aktualisiert."
- note added: "Der Level-Shifter wird von einer Konstantstromquelle bestehend aus Q5 und LED3 gespeist, die der Controller über den Transistor Q3 explizit aktivieren muss."
- note added: "Der mit U5 aufgebaute Differenzverstärker ermittelt den exakten Wert an den Ausgangsspannungsklemmen, teilt ihn durch drei und führt das Ergebnis der Regelschleife zu."
- note added: "Die Leistungsstufe mit Q6 und Q12 sorgt nur für Stromverstärkung. Notbremse" in Form von Q7, die schnelle Überstromimpulse noch vor der Stromregelung abfängt. Steigt die Spannung über dem Widerstand R56 über 1,5 V (gleichbedeutend mit einem Strom von rund 3 A), zieht Q7 die Ausgangsspannung nach unten."
- note added: "Level Shifter Der Regelstufe folgt ein Spannungsumsetzer um Transistor Q4, der den für die gewünschte maximale Ausgangsspannung erforderlichen Spannungshub erzeugt. Q4 arbeitet in (rückgekoppelter) Basisschaltung, da dies schnell ist und weil die Ein- und Ausgangsspannungen dieselbe Phasenlage aufweisen."
- note added: "Liegt beispielsweise an den Klemmen eine Spannung von 30 V an, sind an Pin 1 von U5 genau 10 V zu messen. Die Teilung ist deshalb nötig, weil die Regelschleife nur innerhalb ihrer Betriebsspannung arbeiten kann, und die beträgt hier ±15 V - sehr viel mehr vertragen die OpAmps auch nicht. Wer die Schaltung für höhere Ausgangsspannungen modifizieren möchte, greift am besten hier ein: Je größer die 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"
- note added: "Opto-Bus"
- note added: "U Sensing"
- note added: "Zeitkonstante R19/C13"
- note added: "Zeitkonstante R26/C20"
- moved on the sheet: DCG.C23, DCG.D5, DCG.D6, DCG.D7, DCG.LED3, DCG.PL2, DCG.PL3, DCG.PL6, DCG.PL7, DCG.Q10, DCG.Q11, DCG.Q8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
