File: KiCad/trsmc.kicad_sch (KiCad schematic)
At the start: 48 parts

Commit message: cont. True-RMS Converter
Parts:
- removed TRMSC.C (x4): C, symbol Device:C
- removed TRMSC.C1: 4µ7 50V, symbol Device:C_Polarized
- added TRMSC.C11, TRMSC.C12: 2µ2 MKT, symbol Device:C
- added TRMSC.C2: 4µ7 50V, symbol Device:C_Polarized
- added TRMSC.C3: 100n, symbol Device:C
- added TRMSC.C7: 220n MKT, symbol Device:C
- added TRMSC.JP1, TRMSC.JP2: Jumper_2_Open, symbol Jumper:Jumper_2_Open
- added TRMSC.PL1: (no value), symbol Connector_Generic:Conn_02x08_Odd_Even
- added TRMSC.PL3: AudioJack2, symbol Connector_Audio:AudioJack2
- added TRMSC.PL4: Conn_01x03, symbol Connector_Generic:Conn_01x03
- added TRMSC.PL5: Conn_01x02, symbol Connector_Generic:Conn_01x02
- added TRMSC.R0: 22k lin., symbol Device:R_Potentiometer_Trim
- added TRMSC.R10: 27k, symbol Device:R
- added TRMSC.R11: 47k, symbol Device:R
- added TRMSC.R12, TRMSC.R9: 10k, symbol Device:R
- added TRMSC.R13, TRMSC.R14: 15k, symbol Device:R
- added TRMSC.R15: 22k, symbol Device:R
- added TRMSC.R16: 180k, symbol Device:R
- added TRMSC.R17: 100k, symbol Device:R
- added TRMSC.R21: 4k7, symbol Device:R
- added TRMSC.R32: 470R, symbol Device:R
- added TRMSC.R5: 100k, symbol Device:R_Potentiometer_Trim
- added TRMSC.R6: 5k, symbol Device:R_Potentiometer_Trim
- TRMSC.C10: renamed from TRMSC.C; value C -> SM1206 100n
- TRMSC.C13: renamed from TRMSC.C; value C_Polarized -> 4µ7 25V Ta
Connections:
- net AGnd: now also TRMSC.C10.2, TRMSC.C13.2, TRMSC.U4.1 (GND), TRMSC.U4.6 (OUT_RTN), TRMSC.U4.8 (~{ENABLE}), TRMSC.U5.3 (GND), TRMSC.U6.2 (GND), TRMSC.C11.2, TRMSC.C2.1, TRMSC.C3.2, TRMSC.PL3.S, TRMSC.PL4.1 (Pin_1), TRMSC.R0.1, TRMSC.R13.2, TRMSC.R9.2
- net Attn200: now also TRMSC.PL1.4 (Pin_4)
- net DVcc: now also TRMSC.D4.1 (K), TRMSC.U5.5 (VL), TRMSC.PL1.16 (Pin_16)
- net V+: now also TRMSC.U2.7 (V+), TRMSC.U3.7 (V+), TRMSC.U6.3 (VI), TRMSC.PL1.9 (Pin_9), TRMSC.R5.2
- net V-: now also TRMSC.U2.4 (V-), TRMSC.U3.4 (V-), TRMSC.C2.2, TRMSC.PL1.10 (Pin_10)
- net DVcc-Filtered: now reaches TRMSC.C10.1
- net DVcc-Filtered: now also TRMSC.C13.1, TRMSC.U4.7 (V^{+}), TRMSC.U6.1 (VO), TRMSC.R14.1
- net TRMSC.PL4.E: now reaches TRMSC.U5.1 (D)
- net TRMSC.PL4.E: now also TRMSC.JP2.1 (A), TRMSC.PL4.3 (Pin_3), TRMSC.R0.3
- net Gain10: now reaches TRMSC.U5.6 (IN)
- net Gain10: now also TRMSC.PL1.3 (Pin_3)
- net at TRMSC.U3.2 (-): now also TRMSC.R10.1, TRMSC.R9.1
- net TrueRMS Filtered: now reaches TRMSC.U3.3 (+)
- net TrueRMS Filtered: now also TRMSC.R12.1
- net TP4: now reaches TRMSC.U3.6
- net TP4: now also TRMSC.R11.1, TRMSC.R6.1, TRMSC.R6.2
- net ADC2: now reaches TRMSC.D4.2 (A)
- net ADC2: now also TRMSC.C3.1, TRMSC.PL1.7 (Pin_7), TRMSC.R11.2
- net at TRMSC.U2.1 (VOS): now also TRMSC.R5.1
- net at TRMSC.U2.2 (-): now also TRMSC.R16.1
- net at TRMSC.U2.3 (+): now also TRMSC.R17.2
- net FS_{DC}: now reaches TRMSC.U2.6
- net FS_{DC}: now also TRMSC.C12.1, TRMSC.R12.2, TRMSC.R16.2
- net at TRMSC.U2.8 (VOS): now also TRMSC.R5.3
- net at TRMSC.U4.3 (IN2): now also TRMSC.R13.1, TRMSC.R14.2, TRMSC.R21.2
- net at TRMSC.U4.5 (V_{OUT}): now also TRMSC.C11.1, TRMSC.R15.1
- new net: TRMSC.PL5.2 (Pin_2), TRMSC.R32.1
- new net: TRMSC.C7.2, TRMSC.R21.1
- new net: TRMSC.R10.2, TRMSC.R6.3
- new net ADC3: TRMSC.PL1.8 (Pin_8)
- new net Audio In/Out: TRMSC.JP1.2 (B), TRMSC.PL1.11 (Pin_11), TRMSC.PL3.T
- new net DGnd: TRMSC.PL1.13 (Pin_13), TRMSC.PL1.15 (Pin_15), TRMSC.PL5.1 (Pin_1)
- new net FS_{AC}: TRMSC.C7.1, TRMSC.JP1.1 (A), TRMSC.JP2.2 (B), TRMSC.PL4.2 (Pin_2), TRMSC.R0.2
- new net PC0: TRMSC.PL1.1 (Pin_1)
- new net PC1: TRMSC.PL1.2 (Pin_2)
- new net PC4: TRMSC.PL1.5 (Pin_5), TRMSC.R32.2
- new net PC5: TRMSC.PL1.6 (Pin_6)
- new net TRSMC.PL1.GND: TRMSC.PL1.12 (Pin_12), TRMSC.PL1.14 (Pin_14)
- new net TrueRMS: TRMSC.C12.2, TRMSC.R15.2, TRMSC.R17.1
- no-connect marks 1 -> 3
Other:
- note added: "FS_{2DC} = 2,0V DC"
- note added: "FS_{AC} = 0.5V AC"
- note added: "FS_{DC} = 0,5V DC"
- note added: "SHIELD"
- note added: "T = Tip (Signal) S = Sleeve (GND)"
- moved on the sheet: TRMSC.C, TRMSC.C10, TRMSC.C13, TRMSC.C14, TRMSC.C15, TRMSC.C18, TRMSC.C19, TRMSC.C20, TRMSC.C21, TRMSC.C22, TRMSC.C23, TRMSC.D1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
