File: KiCad/ifp.kicad_sch (KiCad schematic)
At the start: 55 parts, among them U1 FT232RL

Commit message: fixing ifp
Parts:
- added U2: L7915, symbol Regulator_Linear:L7915
- added U3: (no value), symbol ctLab:XPORT
- IFP.C19: value 100 -> 100n
- IFP.U6: value LF411 -> 6N137; footprint Package_DIP:DIP-8_W10.16mm -> Package_DIP:DIP-8_W7.62mm
Connections:
- net AGnd: now also U2.1 (GND)
- net GND: now also IFP.U6.5 (GND), U3.1 (Gnd), U3.9 (Shield); no longer IFP.U6.4 (VCC-)
- net IFP.ETH:TXD: now also U3.4 (Do)
- net IFP.FT232:RXD: now also IFP.U6.6 (VO), U3.5 (Di)
- net IFP.MAX232.RXD: no longer IFP.JP1.1 (A)
- net V--: now also U2.3 (VO)
- net VCC: now also IFP.U6.8 (VCC)
- net RxD_Slave: now reaches IFP.PL2.7 (Pin_7), IFP.PL2.8 (Pin_8)
- net RxD_Slave: now also IFP.U6.3 (C); no longer IFP.U6.1 (B1)
- net at IFP.U6.7 (EN): now also IFP.PL2.3 (Pin_3), IFP.PL2.4 (Pin_4)
- net at IFP.C15.1, IFP.C19.1, IFP.U8.1 (VI): now also U3.2 (Vcc)
- net TxD_Slave: now reaches IFP.PL2.1 (Pin_1), IFP.PL2.2 (Pin_2), IFP.R3.1
- net at IFP.C10.2, IFP.C4.1, IFP.RB1.3 (-): now also U2.2 (VI)
- new net IFP.MAX232:RXD: IFP.JP1.1 (A)
- no-connect marks 29 -> 31
Other:
- moved on the sheet: IFP.C1, IFP.C10, IFP.C11, IFP.C12, IFP.C13, IFP.C16, IFP.C17, IFP.C18, IFP.C2, IFP.C21, IFP.C22, IFP.C23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
