File: KiCad/edl.kicad_sch (KiCad schematic)
At the start: 0 parts

Commit message: Add EDL schematic components
Parts:
- added EDL.C1, EDL.C10, EDL.C2: 22p, Capacitor_THT:C_Disc_D5.0mm_W2.5mm_P2.50mm, symbol Device:C
- added EDL.C11: 47µ 16V, Capacitor_THT:CP_Radial_D6.3mm_P2.50mm, symbol Device:C_Polarized
- added EDL.C12, EDL.C18: 4µ7 35V Ta., Capacitor_THT:CP_Radial_Tantal_D5.0mm_P2.50mm, symbol Device:C_Polarized
- added EDL.C13: 220n, Capacitor_SMD:C_1206_3216Metric, symbol Device:C
- added EDL.C14: 1n, Capacitor_SMD:C_0805_2012Metric, symbol Device:C
- added EDL.C15: 1n, Capacitor_THT:C_Disc_D5.0mm_W2.5mm_P5.00mm, symbol Device:C
- added EDL.C16, EDL.C20, EDL.C22, EDL.C23, EDL.C3, EDL.C5, EDL.C6, EDL.C7, EDL.C8: 100n, Capacitor_THT:C_Disc_D5.0mm_W2.5mm_P5.00mm, symbol Device:C
- added EDL.C17: 10n, Capacitor_THT:C_Disc_D5.0mm_W2.5mm_P5.00mm, symbol Device:C
- added EDL.C19, EDL.C4, EDL.C9: 10µ 35V Ta., Capacitor_THT:CP_Radial_Tantal_D5.0mm_P2.50mm, symbol Device:C_Polarized
- added EDL.C21: 2n2, Capacitor_THT:C_Disc_D5.0mm_W2.5mm_P5.00mm, symbol Device:C
- added EDL.C24: 330n, Capacitor_THT:C_Disc_D5.0mm_W2.5mm_P5.00mm, symbol Device:C
- added EDL.D1, EDL.D2, EDL.D4: 1N4148, Diode_THT:D_DO-35_SOD27_P7.62mm_Horizontal, symbol Diode:1N4148
- added EDL.D3: 1N5401, Diode_THT:D_DO-201AD_P15.24mm_Horizontal, symbol Diode:1N5407
- added EDL.JP1, EDL.JP2, EDL.JP3, EDL.JP4, EDL.JP5: Jumper 2-pol., Connector_PinHeader_2.54mm:PinHeader_1x02_P2.54mm_Vertical, symbol Jumper:Jumper_2_Open
- added EDL.L1: 10µH axial, Inductor_THT:L_Axial_L9.5mm_D4.0mm_P12.70mm_Horizontal_Fastron_SMCC, symbol Device:L_Small
- added EDL.L2: 5µH Stabkerndrossel 3A, Inductor_THT:L_Axial_L20.0mm_D8.0mm_P25.40mm_Horizontal, symbol Device:L_Small
- added EDL.LED1: LED 3mm rot, LED_THT:LED_D3.0mm, symbol Device:LED
- added EDL.PL1: Wannen-Pfostenverbinder 14-pol., Connector_IDC:IDC-Header_2x07_P2.54mm_Vertical, symbol Connector_Generic:Conn_02x07_Odd_Even
- added EDL.PL10, EDL.PL6, EDL.PL7: Platinen-Steckverbinder 2-pol., Connector_PinHeader_2.54mm:PinHeader_1x02_P2.54mm_Vertical, symbol Connector_Generic:Conn_01x02
- added EDL.PL11: Anschlussklemme 4-pol. RM5, TerminalBlock_Altech:Altech_AK100_1x04_P5.00mm, symbol Connector_Generic:Conn_01x04
- added EDL.PL2, EDL.PL3, EDL.PL4, EDL.PL5: Wannen-Pfostenverbinder 10-pol., Connector_IDC:IDC-Header_2x05_P2.54mm_Vertical, symbol Connector_Generic:Conn_02x05_Odd_Even
- added EDL.PL8: Platinen-Steckverbinder 5-pol., Connector_PinHeader_2.54mm:PinHeader_1x05_P2.54mm_Vertical, symbol Connector_Generic:Conn_01x05
- added EDL.PL9: Anschlussklemme 3-pol. RM5, TerminalBlock_Altech:Altech_AK100_1x03_P5.00mm, symbol Connector_Generic:Conn_01x03
- added EDL.Q1, EDL.Q7: BS170, Package_TO_SOT_THT:TO-92_Inline, symbol Transistor_FET:BS170
- added EDL.Q2: BC547B, Package_TO_SOT_THT:TO-92_Inline, symbol Transistor_BJT:BC546
- added EDL.Q3, EDL.Q4: IRFZ44, Package_TO_SOT_THT:TO-220-3_Vertical, symbol Transistor_FET:IRF540N
- added EDL.Q5, EDL.Q6: IRF540, Package_TO_SOT_THT:TO-220-3_Vertical, symbol Transistor_FET:IRF540N
- added EDL.Q8: BC337, Package_TO_SOT_THT:TO-92_Inline, symbol Transistor_BJT:BC546
- added EDL.R1, EDL.R28, EDL.R45, EDL.R49, EDL.R51: 470R, Resistor_THT:R_Axial_DIN0207_L6.3mm_D2.5mm_P10.16mm_Horizontal, symbol Device:R
- added EDL.R10, EDL.R20, EDL.R32, EDL.R34: 10k, Resistor_THT:R_Axial_DIN0207_L6.3mm_D2.5mm_P10.16mm_Horizontal, symbol Device:R
- added EDL.R11, EDL.R14, EDL.R15, EDL.R16, EDL.R17, EDL.R18, EDL.R2, EDL.R3, EDL.R4: 220R, Resistor_THT:R_Axial_DIN0207_L6.3mm_D2.5mm_P10.16mm_Horizontal, symbol Device:R
- added EDL.R12, EDL.R5, EDL.R56, EDL.R59, EDL.R64, EDL.R69: 10R, Resistor_THT:R_Axial_DIN0207_L6.3mm_D2.5mm_P10.16mm_Horizontal, symbol Device:R
- added EDL.R13, EDL.R19, EDL.R55, EDL.R7, EDL.R9: 2k7, Resistor_THT:R_Axial_DIN0207_L6.3mm_D2.5mm_P10.16mm_Horizontal, symbol Device:R
- added EDL.R21, EDL.R22, EDL.R23, EDL.R38, EDL.R40, EDL.R41, EDL.R43, EDL.R47, EDL.R50, EDL.R6: 4k7, Resistor_THT:R_Axial_DIN0207_L6.3mm_D2.5mm_P10.16mm_Horizontal, symbol Device:R
- added EDL.R24, EDL.R30, EDL.R31, EDL.R35, EDL.R42: 1k, Resistor_THT:R_Axial_DIN0207_L6.3mm_D2.5mm_P10.16mm_Horizontal, symbol Device:R
- added EDL.R25, EDL.R26, EDL.R46: 2k2, Resistor_THT:R_Axial_DIN0207_L6.3mm_D2.5mm_P10.16mm_Horizontal, symbol Device:R
- added EDL.R27: R-Array 22kx4, Package_DIP:DIP-8_W7.62mm, symbol Device:R_Pack04
- added EDL.R29, EDL.R54, EDL.R57, EDL.R61, EDL.R62, EDL.R65: 47R, Resistor_THT:R_Axial_DIN0207_L6.3mm_D2.5mm_P10.16mm_Horizontal, symbol Device:R
- added EDL.R33: 30k, Resistor_THT:R_Axial_DIN0207_L6.3mm_D2.5mm_P10.16mm_Horizontal, symbol Device:R
- added EDL.R36, EDL.R53: 220k, Resistor_THT:R_Axial_DIN0207_L6.3mm_D2.5mm_P10.16mm_Horizontal, symbol Device:R
- added EDL.R37: 18k, Resistor_THT:R_Axial_DIN0207_L6.3mm_D2.5mm_P10.16mm_Horizontal, symbol Device:R
- added EDL.R39, EDL.R44, EDL.R48: 2k2 Präz.-Trim. 67X 90°, symbol Device:R_Potentiometer_Trim
- added EDL.R52: 100k, Resistor_THT:R_Axial_DIN0207_L6.3mm_D2.5mm_P10.16mm_Horizontal, symbol Device:R
- added EDL.R58: 680k, Resistor_THT:R_Axial_DIN0207_L6.3mm_D2.5mm_P10.16mm_Horizontal, symbol Device:R
- added EDL.R60: 2k, Resistor_THT:R_Axial_DIN0207_L6.3mm_D2.5mm_P10.16mm_Horizontal, symbol Device:R
- added EDL.R63: 100R, Resistor_THT:R_Axial_DIN0207_L6.3mm_D2.5mm_P10.16mm_Horizontal, symbol Device:R
- added EDL.R66: 0R1 5W, Resistor_THT:R_Axial_Power_L20.0mm_W6.4mm_P25.40mm, symbol Device:R
- added EDL.R67, EDL.R68: 1R 2W, Resistor_THT:R_Axial_DIN0614_L14.3mm_D5.7mm_P20.32mm_Horizontal, symbol Device:R
- added EDL.R8: 0R (Drahtbrücke), Resistor_THT:R_Axial_DIN0207_L6.3mm_D2.5mm_P10.16mm_Horizontal, symbol Device:R
- added EDL.U1: 6N137, Package_DIP:DIP-8_W7.62mm, symbol Isolator:6N137
- added EDL.U10, EDL.U13: OP-27 DIL, Package_DIP:DIP-8_W7.62mm, symbol Amplifier_Operational:OP07
- added EDL.U11, EDL.U8: DG419 DIL, Package_DIP:DIP-8_W7.62mm, symbol CERN:DG419
- added EDL.U12: LF411 DIL, Package_DIP:DIP-8_W7.62mm, symbol ctLab:LF411
- added EDL.U14: LM75 SO8, Package_SO:SOIC-8_3.9x4.9mm_P1.27mm, symbol Sensor_Temperature:LM75C
- added EDL.U2: ATmega32 DIL, Package_DIP:DIP-40_W15.24mm, symbol MCU_Microchip_ATmega:ATmega32-16M
- added EDL.U3: OPA2277 DIL, Package_DIP:DIP-8_W7.62mm, symbol Amplifier_Operational:NE5532
- added EDL.U4: MAX543 DIL / LTC8043 SO8, Package_DIP:DIP-8_W7.62mm, symbol EDL:MAX543_LTC8043
- added EDL.U6: LTC1864 SO8, Package_SO:SOIC-8_3.9x4.9mm_P1.27mm, symbol Analog_ADC:LTC1864
- added EDL.U7: DG409 / DG509 DIL, Package_DIP:DIP-16_W7.62mm, symbol CERN:DG409
- added EDL.U9: LT1019-2.5 DIL, Package_DIP:DIP-8_W7.62mm, symbol Reference_Voltage:LT1019xN8
- added EDL.XTAL1: Quarz 16MHz HC49U, Crystal:Crystal_HC49-U_Vertical, symbol CERN:Quartz Crystal
- added EDL.Z1, EDL.Z3: Z-Diode 5V1 400mW, Diode_THT:D_DO-35_SOD27_P7.62mm_Horizontal, symbol Diode:ZPDxx
- added EDL.Z2: Z-Diode 8V2 400mW, Diode_THT:D_DO-35_SOD27_P7.62mm_Horizontal, symbol Diode:ZPDxx
Connections:
- new net: EDL.U2.17 (VCC), EDL.U2.38 (VCC), EDL.U2.5 (VCC)
- new net: EDL.U2.18 (GND), EDL.U2.39 (GND), EDL.U2.45 (GND), EDL.U2.6 (GND)

Commit message: fixing ifp
Parts:
- removed EDL.U2: ATmega32 DIL, Package_DIP:DIP-40_W15.24mm, symbol MCU_Microchip_ATmega:ATmega32-16M
- added EDL.U2a: ATmega8535-16P, Package_DIP:DIP-40_W15.24mm, symbol MCU_Microchip_ATmega:ATmega8535-16P
- EDL.R8: value 0R (Drahtbrücke) -> 0R
Connections:
- net at EDL.Q8.1 (C): now also EDL.D4.2 (A), EDL.PL10.2 (Pin_2)
- net EDL.Q8.B: now reaches EDL.Q8.2 (B)
- net EDL.Q8.B: now also EDL.R55.2, EDL.U14.3 (O.S.)
- net DGnd: now reaches EDL.Q8.3 (E)
- net DGnd: now also EDL.C1.1, EDL.C2.1, EDL.C23.1, EDL.C3.1, EDL.PL8.3 (Pin_3), EDL.R8.1, EDL.U1.5 (GND), EDL.U1.6 (VO), EDL.U14.4 (GND), EDL.U14.5 (A2), EDL.U14.6 (A1), EDL.U2a.11 (GND)
- net at EDL.JP1.1 (A): now also EDL.PL2.7 (Pin_7), EDL.PL2.8 (Pin_8), EDL.PL3.7 (Pin_7), EDL.PL3.8 (Pin_8)
- net at EDL.JP1.2 (B): now also EDL.PL2.1 (Pin_1), EDL.PL2.2 (Pin_2), EDL.R2.1
- net at EDL.R3.1: now also EDL.PL3.1 (Pin_1), EDL.PL3.2 (Pin_2)
- net at EDL.R3.2: now also EDL.U1.3 (C)
- net AGnd: now reaches EDL.R8.2
- net AGnd: now also EDL.U2a.31 (AGND)
- net EDL.U2a.12: now reaches EDL.C2.2
- net EDL.U2a.12: now also EDL.XTAL1.2 (OSC2)
- net DVcc: now reaches EDL.R55.1
- net DVcc: now also EDL.C23.2, EDL.C3.2, EDL.PL8.2 (Pin_2), EDL.U1.8 (VCC), EDL.U14.7 (A0), EDL.U14.8 (+Vs)
- net at EDL.PL3.10 (Pin_10): now also EDL.JP2.1 (A), EDL.PL2.10 (Pin_10), EDL.PL2.9 (Pin_9), EDL.PL3.9 (Pin_9)
- net at EDL.PL3.3 (Pin_3): now also EDL.PL3.4 (Pin_4), EDL.U1.2 (A)
- net TxD: now reaches EDL.R2.2
- net DVgl+: now reaches EDL.D4.1 (K)
- net DVgl+: now also EDL.PL10.1 (Pin_1), EDL.PL8.1 (Pin_1)
- net PD2: now reaches EDL.LED1.1 (K)
- net at EDL.LED1.2 (A): now also EDL.R1.2
- net RxD: now reaches EDL.U1.7 (EN)
- net I2C_SDA: now reaches EDL.U14.1 (SDA)
- net I2C_SDA: now also EDL.PL8.4 (Pin_4)
- net I2C_SCL: now reaches EDL.U14.2 (SCL)
- net I2C_SCL: now also EDL.PL8.5 (Pin_5)
- net at EDL.R1.1: now also EDL.JP2.2 (B), EDL.PL2.3 (Pin_3), EDL.PL2.4 (Pin_4)
- net EDL.U2a.13: now reaches EDL.C1.2
- net EDL.U2a.13: now also EDL.XTAL1.1 (OSC1)
- no-connect marks 0 -> 4
Other:
- moved on the sheet: EDL.PL8, EDL.Q8, EDL.U14

Commit message: cont. eld
Parts:
- added EDL.ADC16: Conn_01x01_Socket, symbol Connector:Conn_01x01_Socket
- added EDL.LQ3, EDL.LQ4, EDL.LQ5, EDL.LQ6, EDL.LQ7: ${VALUE}, symbol CERN:Ferrite Bead
Connections:
- net PD2 is gone; now on net ADC1: EDL.LED1.1 (K)
- net RxD is gone; now on net PD0: EDL.U1.7 (EN)
- net TxD is gone; now on net PD1: EDL.R2.2
- net AGnd: now also EDL.C11.2, EDL.C12.2, EDL.C13.1, EDL.C14.1, EDL.C8.1, EDL.C9.2, EDL.U6.3 (IN^{-}), EDL.U6.4 (GND), EDL.U7.15 (GND), EDL.U9.4 (GND), EDL.Z1.2 (A)
- net DGnd: now also EDL.JP3.1 (A), EDL.JP4.1 (A), EDL.JP5.1 (A), EDL.PL4.10 (Pin_10), EDL.PL4.4 (Pin_4), EDL.PL4.6 (Pin_6), EDL.PL4.8 (Pin_8), EDL.PL5.7 (Pin_7), EDL.PL5.9 (Pin_9), EDL.PL6.2 (Pin_2), EDL.PL7.2 (Pin_2)
- net DVcc: now also EDL.L1.2, EDL.PL4.2 (Pin_2), EDL.PL5.10 (Pin_10), EDL.PL5.8 (Pin_8), EDL.R10.1, EDL.R13.1, EDL.R19.1, EDL.R6.1, EDL.R7.1, EDL.R9.1, EDL.U2a.30 (AVCC)
- net I2C_SCL: now also EDL.PL5.6 (Pin_6), EDL.R9.2, EDL.U2a.22 (PC0)
- net I2C_SDA: now also EDL.PL5.5 (Pin_5), EDL.R13.2, EDL.U2a.23 (PC1)
- net TP2: now reaches EDL.Z1.1 (K)
- net TP2: now also EDL.R20.1, EDL.R37.1, EDL.R42.2, EDL.R45.1, EDL.U11.8 (S2)
- net PD0: now reaches EDL.R7.2
- net PD0: now also EDL.U2a.14 (PD0)
- net EDL.PL6:TTL: now reaches EDL.PL6.1 (Pin_1)
- net EDL.PL6:TTL: now also EDL.R10.2, EDL.R4.1
- net at EDL.Q6.1 (G): now also EDL.R65.1
- net Drain Ext.: now reaches EDL.Q6.2 (D)
- net Drain Ext.: now also EDL.Q3.2 (D), EDL.Q4.2 (D), EDL.Q5.2 (D), EDL.Q7.1 (D)
- net at EDL.Q6.3 (S): now also EDL.LQ6.2
- net GNDD: now reaches EDL.R52.2
- net GNDD: now also EDL.C16.1, EDL.C17.1, EDL.C19.2, EDL.C22.1, EDL.C4.2, EDL.C7.1, EDL.Q1.3 (S), EDL.Q2.3 (E), EDL.Z2.2 (A), EDL.Z3.2 (A)
- net at EDL.R63.1: now also EDL.LQ7.1
- net OC1A: now reaches EDL.JP3.2 (B)
- net OC1A: now also EDL.U2a.19 (PD5)
- net at EDL.R61.1: now also EDL.Q5.1 (G)
- net at EDL.Q2.1 (C): now also EDL.D1.1 (K)
- net SDATAIN1_R: now reaches EDL.R19.2
- net SDATAIN1_R: now also EDL.R17.2, EDL.U6.6 (SDO)
- net at EDL.R35.1: now also EDL.ADC16.1 (Pin_1)
- net at EDL.R35.2: now also EDL.C14.2, EDL.R36.2, EDL.U6.2 (IN^{+})
- net ADC0: now reaches EDL.PL5.1 (Pin_1)
- net ADC0: now also EDL.U2a.40 (PA0)
- net ADC1: now reaches EDL.PL5.2 (Pin_2)
- net ADC1: now also EDL.PL5.3 (Pin_3), EDL.U2a.16 (PD2), EDL.U2a.39 (PA1)
- net INT1: now reaches EDL.PL5.4 (Pin_4)
- net INT1: now also EDL.U2a.17 (PD3)
- net INT2: now reaches EDL.R4.2
- net INT2: now also EDL.U2a.3 (PB2)
- net at EDL.R64.1: now also EDL.LQ6.1
- net DVcc_ADC: now reaches EDL.U9.2 (IN)
- net DVcc_ADC: now also EDL.C11.1, EDL.C13.2, EDL.C8.2, EDL.L1.1, EDL.U2a.10 (VCC), EDL.U6.8 (V_{CC})
- net ARef: now reaches EDL.U9.6 (OUT)
- net ARef: now also EDL.C9.1, EDL.R36.1, EDL.U2a.32 (AREF), EDL.U6.1 (V_{REF})
- net at EDL.Q7.2 (G): now also EDL.R62.1
- net at EDL.Q7.3 (S): now also EDL.LQ7.2
- net Gate Ext.: now reaches EDL.R54.1
- net Gate Ext.: now also EDL.R57.1
- net at EDL.R54.2: now also EDL.Q3.1 (G)
- net V+: now reaches EDL.C12.1
- net V+: now also EDL.U7.14 (V+)
- net OC2: now reaches EDL.JP5.2 (B)
- net OC2: now also EDL.U2a.21 (PD7)
- net PC2: now reaches EDL.U7.1 (A0)
- net PC2: now also EDL.U2a.24 (PC2)
- net EDL.U7:S4B: now reaches EDL.U7.10 (S4B)
- net EDL.U7:S3B: now reaches EDL.U7.11 (S3B)
- net EDL.U7:S2B: now reaches EDL.U7.12 (S2B)
- net EDL.U7:S1B: now reaches EDL.U7.13 (S1B)
- net PC3: now reaches EDL.U7.16 (A1)
- net PC3: now also EDL.U2a.25 (PC3)
- net PC4: now reaches EDL.U7.2 (EN)
- net PC4: now also EDL.U2a.26 (PC4)
- net V-: now reaches EDL.U7.3 (V-)
- net EDL.U7:S1A: now reaches EDL.U7.4 (S1A)
- net EDL.U7:S2A: now reaches EDL.U7.5 (S2A)
- net EDL.U7:S3A: now reaches EDL.U7.6 (S3A)
- net EDL.U7:S4A: now reaches EDL.U7.7 (S4A)
- net EDL.U7:DA: now reaches EDL.U7.8 (DA)
- net EDL.U7:DA: now also EDL.D1.2 (A)
- net EDL.U7:DB: now reaches EDL.U7.9 (DB)
- net EDL.PL7:TTL: now reaches EDL.PL7.1 (Pin_1)
- net EDL.PL7:TTL: now also EDL.R11.2
- net ICP: now reaches EDL.JP4.2 (B)
- net ICP: now also EDL.U2a.20 (PD6)
- net at EDL.R68.1: now also EDL.LQ5.1
- net at EDL.Q3.3 (S): now also EDL.LQ3.2
- net PB4: now reaches EDL.R16.1
- net PB4: now also EDL.U2a.5 (PB4)
- net STRAD24_R: now reaches EDL.R16.2
- net STRAD24_R: now also EDL.U6.5 (CONV)
- net at EDL.Q5.3 (S): now also EDL.LQ5.2
- net SCLK_R: now reaches EDL.U6.7 (SCK)
- net SCLK_R: now also EDL.R18.2
- net PB0: now reaches EDL.U2a.1 (PB0)
- net EDL.U2a.XTAL2: now reaches EDL.U2a.12 (XTAL2)
- net EDL.U2a.XTAL1: now reaches EDL.U2a.13 (XTAL1)
- net PD1: now reaches EDL.U2a.15 (PD1)
- net OC1B: now reaches EDL.U2a.18 (PD4)
- net PB1: now reaches EDL.U2a.2 (PB1)
- net PC5: now reaches EDL.U2a.27 (PC5)
- net PC6: now reaches EDL.U2a.28 (PC6)
- net PC7: now reaches EDL.U2a.29 (PC7)
- net PC7: now also EDL.R11.1
- net ADC7: now reaches EDL.U2a.33 (PA7)
- net ADC6: now reaches EDL.U2a.34 (PA6)
- net ADC5: now reaches EDL.U2a.35 (PA5)
- net ADC4: now reaches EDL.U2a.36 (PA4)
- net ADC3: now reaches EDL.U2a.37 (PA3)
- net ADC2: now reaches EDL.U2a.38 (PA2)
- net OC0: now reaches EDL.U2a.4 (PB3)
- net MOSI: now reaches EDL.U2a.6 (PB5)
- net MOSI: now also EDL.PL4.1 (Pin_1)
- net MISO: now reaches EDL.U2a.7 (PB6)
- net MISO: now also EDL.PL4.9 (Pin_9), EDL.R17.1
- net PB7: now reaches EDL.U2a.8 (PB7)
- net PB7: now also EDL.PL4.7 (Pin_7), EDL.R18.1
- net Reset: now reaches EDL.U2a.9 (~{RESET})
- net Reset: now also EDL.PL4.5 (Pin_5), EDL.R6.2
- net at EDL.R66.1: now also EDL.LQ3.1, EDL.LQ4.1
- net at EDL.Q4.1 (G): now also EDL.R57.2
- net at EDL.Q4.3 (S): now also EDL.LQ4.2
- net EDL.Q8.B renamed EDL.Q8:B
- net EDL.U2a.12 renamed EDL.U2a:XTAL2
- net EDL.U2a.13 renamed EDL.U2a:XTAL1
- no-connect marks 4 -> 9
Other:
- moved on the sheet: EDL.C1, EDL.C2, EDL.C23, EDL.C3, EDL.D4, EDL.JP1, EDL.JP2, EDL.LED1, EDL.PL10, EDL.PL2, EDL.PL3, EDL.PL8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

Commit message: finishing edl schematic
Parts:
- removed EDL.ADC16: Conn_01x01_Socket, symbol Connector:Conn_01x01_Socket
- removed EDL.L2: 5µH Stabkerndrossel 3A, Inductor_THT:L_Axial_L20.0mm_D8.0mm_P25.40mm_Horizontal, symbol Device:L_Small
- added EDL.L2: 5µH 3A, symbol Device:L_Ferrite
- EDL.PL11: value Anschlussklemme 4-pol. RM5 -> (none)
- EDL.R39, EDL.R44, EDL.R48: value 2k2 Präz.-Trim. 67X 90° -> 2k2
- EDL.Z2: value Z-Diode 8V2 400mW -> 8V2 400mW
Connections:
- net Gate Ext. is gone; now on net EDL.U7:S1A: EDL.R54.1, EDL.R57.1
- net ADC2: now also EDL.C5.2, EDL.R34.2
- net ADC3: now also EDL.C6.2, EDL.R20.2
- net AGnd: now also EDL.C18.2, EDL.C20.2, EDL.C5.1, EDL.C6.1, EDL.PL1.7 (Pin_7), EDL.PL1.8 (Pin_8), EDL.PL11.3 (Pin_3), EDL.R24.2, EDL.R25.2, EDL.R26.2, EDL.R56.2, EDL.R60.2, EDL.U11.3 (GND), EDL.U4.4 (GND), EDL.U8.3 (GND)
- net ARef: now also EDL.R34.1, EDL.U8.8 (S2)
- net DGnd: now also EDL.PL1.11 (Pin_11), EDL.PL1.12 (Pin_12), EDL.PL1.3 (Pin_3), EDL.PL1.4 (Pin_4)
- net DVcc: now also EDL.PL1.13 (Pin_13), EDL.PL1.14 (Pin_14)
- net DVcc_ADC: now also EDL.C18.1, EDL.U11.5 (VL), EDL.U4.8 (VDD), EDL.U8.5 (VL)
- net DVgl+: now also EDL.PL1.1 (Pin_1), EDL.PL1.2 (Pin_2)
- net Drain Ext.: now also EDL.PL9.2 (Pin_2), EDL.R67.1, EDL.L2.1
- net EDL.U7:DA: now also EDL.R28.2, EDL.Z2.1 (K)
- net EDL.U7:DB: now also EDL.R46.2
- net EDL.U7:S1A: now also EDL.PL9.1 (Pin_1), EDL.R27.5 (R4.2)
- net EDL.U7:S2A: now also EDL.R27.6 (R3.2), EDL.R61.2
- net EDL.U7:S3A: now also EDL.R27.7 (R2.2), EDL.R65.2
- net EDL.U7:S4A: now also EDL.R27.8 (R1.2), EDL.R62.2
- net GNDD: now also EDL.C4.1; no longer EDL.C4.2
- net MOSI: now also EDL.R15.1
- net OC0: now also EDL.R14.1
- net PB0: now also EDL.U8.6 (IN)
- net PB1: now also EDL.U11.6 (IN)
- net PC5: now also EDL.Q1.2 (G)
- net SCLK_R: now also EDL.U4.7 (CLK)
- net TP2: now also EDL.R42.1, EDL.R45.2; no longer EDL.R42.2, EDL.R45.1
- net V+: now also EDL.C16.2, EDL.C19.1, EDL.C22.2, EDL.R12.2, EDL.R39.2, EDL.R48.2, EDL.U10.7 (V+), EDL.U11.4 (V+), EDL.U12.7 (VCC+), EDL.U13.7 (V+), EDL.U3.8 (V+), EDL.U8.4 (V+)
- net V-: now also EDL.C20.1, EDL.C4.2, EDL.C7.2, EDL.R23.2, EDL.R5.2, EDL.U10.4 (V-), EDL.U11.7 (V-), EDL.U13.4 (V-), EDL.U3.4 (V-), EDL.U8.7 (V-)
- net at EDL.R38.1: now also EDL.R48.1
- net EDL.U13:1: now reaches EDL.R38.2
- net EDL.U13:1: now also EDL.U13.1 (VOS)
- net V--: now reaches EDL.PL1.10 (Pin_10)
- net V--: now also EDL.PL1.9 (Pin_9), EDL.R5.1
- net V++: now reaches EDL.PL1.5 (Pin_5)
- net V++: now also EDL.PL1.6 (Pin_6), EDL.R12.1
- net at EDL.R37.2: now also EDL.R60.1, EDL.U13.2 (-)
- net at EDL.R52.1: now also EDL.R53.1, EDL.U12.3 (In+)
- net TP1: now reaches EDL.R33.1
- net TP1: now also EDL.R49.2, EDL.U11.2 (S1), EDL.Z3.1 (K)
- net at EDL.R33.2: now also EDL.R32.1, EDL.U12.2 (In-)
- net at EDL.R43.1: now also EDL.U12.1 (B1)
- net at EDL.R43.2: now also EDL.R44.3
- net PwrGnd: now reaches EDL.C24.1
- net PwrGnd: now also EDL.D3.2 (A), EDL.PL11.4 (Pin_4), EDL.R56.1, EDL.R63.2, EDL.R64.2, EDL.R66.2, EDL.R68.2
- net at EDL.C24.2: now also EDL.R69.2
- net at EDL.R39.1: now also EDL.R40.2
- net at EDL.R39.3: now also EDL.R41.2
- net at EDL.R49.1: now also EDL.U12.6 (OUT)
- net EDL.ADC16: now reaches EDL.R35.1
- net EDL.ADC16: now also EDL.U11.1 (D)
- net EDL.U10:OUT: now reaches EDL.D2.1 (K)
- net EDL.U10:OUT: now also EDL.R28.1, EDL.R51.2, EDL.U10.6
- net EDL.U10:IN-: now reaches EDL.D2.2 (A)
- net EDL.U10:IN-: now also EDL.C21.2, EDL.R42.2, EDL.U10.2 (-)
- net EDL.U10:1: now reaches EDL.R41.1
- net EDL.U10:1: now also EDL.U10.1 (VOS)
- net at EDL.R51.1: now also EDL.C21.1
- net SDATA_R: now reaches EDL.R15.2
- net SDATA_R: now also EDL.U4.6 (SRI)
- net EDL.U10:8: now reaches EDL.R40.1
- net EDL.U10:8: now also EDL.U10.8 (VOS)
- net VRef: now reaches EDL.U8.1 (D)
- net RmodeRef: now reaches EDL.U8.2 (S1)
- net EDL.U13:8: now reaches EDL.R47.1
- net EDL.U13:8: now also EDL.U13.8 (VOS)
- net at EDL.R47.2: now also EDL.R48.3
- net at EDL.R24.1: now also EDL.R23.1, EDL.R27.1 (R1.1), EDL.R27.2 (R2.1), EDL.R27.3 (R3.1), EDL.R27.4 (R4.1)
- net at EDL.R26.1: now also EDL.U3.5 (+)
- net at EDL.R67.2: now also EDL.R59.1, EDL.L2.2
- net at EDL.U13.3 (+): now also EDL.C15.1, EDL.R30.2, EDL.R46.1
- net at EDL.U13.6: now also EDL.R45.1
- net at EDL.R32.2: now also EDL.Q1.1 (D)
- net Vref: now reaches EDL.U4.1 (VREF)
- net Rfb: now reaches EDL.U4.2 (RFB)
- net Rfb: now also EDL.C10.1, EDL.R21.1, EDL.U3.1
- net DACout: now reaches EDL.U4.3 (IOUT)
- net DACout: now also EDL.C10.2, EDL.U3.2 (-)
- net STRDAC_R: now reaches EDL.U4.5 (~{LOAD})
- net STRDAC_R: now also EDL.R14.2
- net at EDL.R25.1: now also EDL.U3.3 (+)
- net at EDL.U3.6 (-): now also EDL.R21.2, EDL.R22.1
- net at EDL.U3.7: now also EDL.R22.2, EDL.R31.1
- net at EDL.C15.2: now also EDL.R29.2
- net EDL.PL11:In+: now reaches EDL.R69.1
- net EDL.PL11:In+: now also EDL.D3.1 (K), EDL.PL11.1 (Pin_1)
- net Source Ext.: now reaches EDL.PL9.3 (Pin_3)
- net at EDL.R44.1: now also EDL.R50.2
- net at EDL.R44.2: now also EDL.U12.4 (VCC-)
- net at EDL.R29.1: now also EDL.Q2.2 (B), EDL.R30.1
- net EDL.U10:IN+: now reaches EDL.C17.2
- net EDL.U10:IN+: now also EDL.R31.2, EDL.U10.3 (+)
- net at EDL.R53.2: now also EDL.R58.2
- net EDL.PL11:Sense In+: now reaches EDL.R58.1
- net EDL.PL11:Sense In+: now also EDL.PL11.2 (Pin_2), EDL.R59.2
- net at EDL.U12.5 (B2): now also EDL.R50.1
Other:
- moved on the sheet: EDL.C1, EDL.C11, EDL.C12, EDL.C13, EDL.C14, EDL.C2, EDL.C23, EDL.C3, EDL.C8, EDL.C9, EDL.D1, EDL.D4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

Commit message: cont. div
Other:
- title: (none) -> Elektronische Last (EDL)
Changed lines of the file:
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@@
 	(generator_version "10.0")
 	(paper "A0")
+	(title_block
+		(title "Elektronische Last (EDL)")
+		(comment 1 "ct.08.12.176-181")
+	)
 	(junction
 		(at 212.09 331.47)
