File: KiCad/div.kicad_sch (KiCad schematic)
At the start: 97 parts

Commit message: starting DIV
Parts:
- removed DIV.SW2, DIV.SW3, DIV.SW4, DIV.SW5, DIV.SW6: Min.-Relais 2-pol. um 12V (Omron G5V-2 / SDS DS2E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, Relay_THT:Relay_DPDT_Omron_G5V-2, symbol Relay:Relay_DPDT
- removed DIV.U9: ULN2003 / ULN2803 DIL, Package_DIP:DIP-16_W7.62mm, symbol Transistor_Array:ULN2003
- added DIV.SW2, DIV.SW3, DIV.SW4, DIV.SW5, DIV.SW6: Omron G5V-2 / SDS DS2E-M-DC12V, symbol ctLab:G5V-2
- added DIV.U9: UNL2803, Package_DIP:DIP-16_W10.16mm, symbol ctLab:ULN2803A
- DIV.PL1: value Wannen-Pfostenverbinder 14-pol. -> Power Supply
- DIV.U8: value LM399 (siehe Text) -> LM399
Connections:
- net DVgl+: now reaches DIV.C4.1
- net DVgl+: now also DIV.PL1.1 (Pin_1), DIV.PL1.2 (Pin_2), DIV.SW2.1 (A1), DIV.SW3.1 (A1), DIV.SW4.1 (A1), DIV.SW5.1 (A1), DIV.SW6.1 (A1), DIV.U9.10 (COM)
- net DGnd: now reaches DIV.C4.2
- net DGnd: now also DIV.PL1.11 (Pin_11), DIV.PL1.12 (Pin_12), DIV.PL1.3 (Pin_3), DIV.PL1.4 (Pin_4), DIV.U9.9 (GND)
- net V--: now reaches DIV.PL1.10 (Pin_10)
- net V--: now also DIV.PL1.9 (Pin_9)
- net DVcc: now reaches DIV.PL1.13 (Pin_13)
- net DVcc: now also DIV.PL1.14 (Pin_14)
- net V++: now reaches DIV.PL1.5 (Pin_5)
- net V++: now also DIV.PL1.6 (Pin_6)
- net AGnd: now reaches DIV.PL1.7 (Pin_7)
- net AGnd: now also DIV.PL1.8 (Pin_8)
- new net DIV.U9.OUT2: DIV.SW3.16 (A2), DIV.U9.17 (OUT2)
- new net DIV.U9.OUT3: DIV.SW2.16 (A2), DIV.U9.16 (OUT3)
- new net DIV.U9.OUT4: DIV.SW6.16 (A2), DIV.U9.15 (OUT4)
- new net DIV.U9.OUT5: DIV.SW4.16 (A2), DIV.U9.14 (OUT5)
- new net DIV.U9.OUT6: DIV.SW5.16 (A2), DIV.U9.13 (OUT6)
- new net DIV.U9.OUT7: DIV.U9.12 (OUT7)
- new net DIV.U9.OUT8: DIV.U9.11 (OUT8)
- new net PA5: DIV.U9.4 (IN4)
- new net PA6: DIV.U9.3 (IN3)
- new net PA7: DIV.U9.2 (IN2)
- new net PC4: DIV.U9.8 (IN8)
- new net PC5: DIV.U9.7 (IN7)
- new net PC6: DIV.U9.6 (IN6)
- new net PC7: DIV.U9.5 (IN5)
- no-connect marks 0 -> 2
Other:
- moved on the sheet: DIV.C1, DIV.C10, DIV.C11, DIV.C12, DIV.C13, DIV.C14, DIV.C16, DIV.C17, DIV.C2, DIV.C3, DIV.C5, DIV.C6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

Commit message: cont. div
Parts:
- added DIV.SW1, DIV.SW7: HE721A0500, symbol ctLab:HE721A0500
- DIV.FS1: value Sicherung 2,5A FF mit Halter -> 2,5A FF; Description1 (none) -> Sicherung mit Halter
- DIV.HV1: value EC350X Epcos B88069X0810S102 -> EC350X; Description:1 (none) -> Epcos B88069X0810S102
- DIV.PL7: value Platinen-Steckverbinder 2-pol. -> (none); Description:1 (none) -> Platinen-Steckverbinder 2-pol.; Description:2 (none) -> TRSMC Input
- DIV.PL8, DIV.PL9: value Anschlussklemme 2-pol. RM5 -> (none); Description:1 (none) -> Anschlussklemme 2-pol. RM5
- DIV.R38: value 0,1R 1%, Isabellenhütte RM20/RM27,5 -> 0,1R 1%; Description:1 (none) -> Isabellenhütte RM20/RM27,5
- DIV.R39: value 9M 0,1%, RM20 -> 9M 0,1% RM20
Connections:
- net AGnd: now also DIV.C17.2, DIV.D3.2 (A), DIV.D4.1 (K), DIV.HV1.1, DIV.PL7.1 (Pin_1), DIV.PL8.2 (Pin_2), DIV.PL9.2 (Pin_2), DIV.R34.2, DIV.R35.2, DIV.R36.2, DIV.R38.2
- net DVcc: now also DIV.SW1.2 (A2), DIV.SW7.2 (A2)
- net V++: now also DIV.R5.1
- net V--: now also DIV.R6.1
- net at DIV.R28.1: now also DIV.R33.2
- net DIV.U6:IN+: now reaches DIV.R28.2
- net DIV.U6:IN+: now also DIV.C17.1, DIV.SW1.[1,14] (12), DIV.SW7.[1,14] (12)
- net DIV.SW4:Pin13: now reaches DIV.FS1.1
- net DIV.SW4:Pin13: now also DIV.HV1.3, DIV.SW4.13 (2)
- net Input: now reaches DIV.FS1.2
- net Input: now also DIV.PL9.1 (Pin_1)
- net DIV.SW3:Pin9: now reaches DIV.R38.1
- net DIV.SW3:Pin9: now also DIV.PL8.1 (Pin_1), DIV.SW3.9 (21)
- net at DIV.D4.2 (A): now also DIV.D2.1 (K)
- net V+: now reaches DIV.R5.2
- net at DIV.R34.1: now also DIV.SW2.9 (21)
- net at DIV.R37.1: now also DIV.R39.2, DIV.SW7.[7,8] (1)
- net at DIV.R37.2: now also DIV.R36.1, DIV.SW1.[7,8] (1)
- net at DIV.SW5.11 (22): now also DIV.SW5.6 (12)
- net at DIV.SW5.13 (2): now also DIV.SW6.4 (1)
- net at DIV.SW5.4 (1): now also DIV.SW4.11 (22), DIV.SW4.8 (11)
- net AC: now reaches DIV.SW5.8 (11)
- net AC: now also DIV.PL7.2 (Pin_2)
- net TRMS: now reaches DIV.SW5.9 (21)
- net at DIV.SW6.6 (12): now also DIV.R33.1
- net at DIV.SW6.8 (11): now also DIV.R39.1
- net V-: now reaches DIV.R6.2
- net at DIV.R35.1: now also DIV.SW2.11 (22)
- net at DIV.D3.1 (K): now also DIV.D1.2 (A)
- net DIV.SW3:Pin11: now reaches DIV.D2.2 (A)
- net DIV.SW3:Pin11: now also DIV.D1.1 (K), DIV.SW2.13 (2), DIV.SW3.11 (22)
- net DIV.SW3:Pin13: now reaches DIV.SW3.13 (2)
- net DIV.SW3:Pin13: now also DIV.SW4.9 (21)
- net at DIV.SW3.4 (1): now also DIV.SW2.6 (12)
- net at DIV.SW2.4 (1): now also DIV.SW4.4 (1)
- net DIV.U9.OUT2 renamed DIV.U9:OUT2
- net DIV.U9.OUT3 renamed DIV.U9:OUT3
- net DIV.U9.OUT4 renamed DIV.U9:OUT4
- net DIV.U9.OUT5 renamed DIV.U9:OUT5
- net DIV.U9.OUT6 renamed DIV.U9:OUT6
- net DIV.U9.OUT7 renamed DIV.U9:OUT7
- net DIV.U9:OUT7: now also DIV.SW1.6 (A1)
- net DIV.U9.OUT8 renamed DIV.U9:OUT8
- net DIV.U9:OUT8: now also DIV.SW7.6 (A1)
- no-connect marks 2 -> 4
Other:
- note added: "Buffer IN"
- title: DIV Component Inventory -> Digital Voltmeter (DIV)
- moved on the sheet: DIV.SW2, DIV.SW3, DIV.SW4, DIV.SW5, DIV.SW6

Commit message: improving div schematic
Parts:
- DIV.M1: value Wannen-Pfostenverbinder 16-pol. (TRMSC-Modul) -> (none); Description:1 (none) -> TRMSC; Description:2 (none) -> Wannen-Pfostenverbinder 16-pol.
- DIV.PL2: value Wannen-Pfostenverbinder 10-pol. -> (none); Description:0 (none) -> Wannen-Pfostenverbinder 10-pol.; Description:1 (none) -> OptoOut
- DIV.PL3: value Wannen-Pfostenverbinder 10-pol. -> (none); Description:0 (none) -> Wannen-Pfostenverbinder 10-pol.; Description:1 (none) -> OptoIn
- DIV.PL4: value Wannen-Pfostenverbinder 10-pol. -> (none); Description:0 (none) -> Wannen-Pfostenverbinder 10-pol.; Description:1 (none) -> ISP
- DIV.PL5: value Wannen-Pfostenverbinder 10-pol. -> (none); Description:0 (none) -> Wannen-Pfostenverbinder 10-pol.; Description:1 (none) -> Panel
- DIV.R13: value 10k Präz.-Trimmer W64 (siehe Text) -> 10k; Description:1 (none) -> Präz.-Trimmer W64
- DIV.SW5: Descripton1 AC -> DC/AC
- DIV.U3: value LT1019 / REF-43 DIL -> LT1019 or REF-43 DIL
Connections:
- net DIV.SW3:Pin9 is gone; now on net In 10A: DIV.PL8.1 (Pin_1), DIV.R38.1, DIV.SW3.9 (21)
- net TRMS is gone; now on net PA2: DIV.SW5.9 (21)
- net AGnd: now also DIV.C10.1, DIV.C12.2, DIV.C6.1, DIV.C8.2, DIV.M1.12 (Pin_12), DIV.M1.14 (Pin_14), DIV.R19.2, DIV.U1.31 (AGND), DIV.U3.4 (GND), DIV.U7.3 (GND)
- net DGnd: now also DIV.JP3.1 (A), DIV.JP4.1 (A), DIV.JP5.1 (A), DIV.M1.13 (Pin_13), DIV.M1.15 (Pin_15), DIV.PL4.10 (Pin_10), DIV.PL4.4 (Pin_4), DIV.PL4.6 (Pin_6), DIV.PL4.8 (Pin_8), DIV.PL5.7 (Pin_7), DIV.PL5.9 (Pin_9), DIV.PL6.1 (Pin_1)
- net DVcc: now also DIV.C3.1, DIV.L1.1, DIV.M1.16 (Pin_16), DIV.PL4.2 (Pin_2), DIV.PL5.10 (Pin_10), DIV.PL5.8 (Pin_8), DIV.R1.2, DIV.R14.1, DIV.R16.1, DIV.R24.2, DIV.R7.1, DIV.U1.10 (VCC), DIV.U2.8 (VCC), DIV.U7.5 (VL)
- net PA5: now also DIV.U1.35 (PA5)
- net PA6: now also DIV.U1.34 (PA6)
- net PA7: now also DIV.U1.33 (PA7)
- net PC4: now also DIV.M1.5 (Pin_5), DIV.U1.26 (PC4)
- net PC5: now also DIV.M1.6 (Pin_6), DIV.U1.27 (PC5)
- net PC6: now also DIV.U1.28 (PC6)
- net PC7: now also DIV.U1.29 (PC7)
- net V+: now also DIV.M1.9 (Pin_9), DIV.Q2.1 (C), DIV.U6.7 (VCC+), DIV.U7.4 (V+)
- net V-: now also DIV.C10.2, DIV.C6.2, DIV.M1.10 (Pin_10), DIV.Q1.2 (B), DIV.Q1.3 (E), DIV.R13.2, DIV.U6.4 (VCC-), DIV.U7.7 (V-)
- net at DIV.R13.1: now also DIV.U6.1 (B1)
- net at DIV.R13.3: now also DIV.U6.5 (B2)
- net at DIV.R35.1, DIV.SW2.11 (22): now also DIV.SW3.6 (12)
- net DVcc-ADC: now reaches DIV.C12.1
- net DVcc-ADC: now also DIV.C8.1, DIV.L1.2, DIV.U1.30 (AVCC), DIV.U3.2 (IN)
- net DCmid: now reaches DIV.C11.1
- net DCmid: now also DIV.R20.1, DIV.U6.6 (OUT), DIV.U7.2 (S1)
- net at DIV.C11.2: now also DIV.R19.1, DIV.R20.2, DIV.U7.8 (S2)
- net ICP: now reaches DIV.JP4.2 (B)
- net ICP: now also DIV.U1.20 (PD6)
- net at DIV.PL3.1 (Pin_1): now also DIV.PL3.2 (Pin_2), DIV.R3.1
- net at DIV.PL3.10 (Pin_10): now also DIV.JP2.1 (A), DIV.PL2.10 (Pin_10), DIV.PL2.9 (Pin_9), DIV.PL3.9 (Pin_9)
- net at DIV.PL3.3 (Pin_3): now also DIV.PL3.4 (Pin_4), DIV.U2.2 (A)
- net at DIV.PL3.7 (Pin_7): now also DIV.JP1.1 (A), DIV.PL2.7 (Pin_7), DIV.PL2.8 (Pin_8), DIV.PL3.8 (Pin_8)
- net at DIV.U2.3 (C): now also DIV.R3.2
- net Gnd: now reaches DIV.U2.5 (GND)
- net Gnd: now also DIV.C1.2, DIV.C2.2, DIV.C3.2, DIV.U1.11 (GND), DIV.U2.6 (VO)
- net PD0: now reaches DIV.U2.7 (EN)
- net PD0: now also DIV.R24.1, DIV.U1.14 (PD0)
- net at DIV.U7.1 (D): now also DIV.U6.2 (In-)
- net OC1B: now reaches DIV.U7.6 (IN)
- net OC1B: now also DIV.U1.18 (PD4)
- net PC0: now reaches DIV.M1.1 (Pin_1)
- net PC0: now also DIV.PL5.6 (Pin_6), DIV.R14.2, DIV.U1.22 (PC0)
- net Audio: now reaches DIV.M1.11 (Pin_11)
- net PC1: now reaches DIV.M1.2 (Pin_2)
- net PC1: now also DIV.PL5.5 (Pin_5), DIV.R16.2, DIV.U1.23 (PC1)
- net Gain10: now reaches DIV.M1.3 (Pin_3)
- net Gain10: now also DIV.U1.24 (PC2)
- net Attn200: now reaches DIV.M1.4 (Pin_4)
- net Attn200: now also DIV.U1.25 (PC3)
- net PA2: now reaches DIV.M1.7 (Pin_7)
- net PA2: now also DIV.U1.38 (PA2)
- net PA3: now reaches DIV.M1.8 (Pin_8)
- net PA3: now also DIV.U1.37 (PA3)
- net at DIV.R34.1, DIV.SW2.9 (21): now also DIV.SW2.8 (11)
- net at DIV.JP2.2 (B): now also DIV.PL2.3 (Pin_3), DIV.PL2.4 (Pin_4)
- net DIV.U6:In+: now reaches DIV.Q2.2 (B)
- net DIV.U6:In+: now also DIV.Q1.1 (C), DIV.Q2.3 (E), DIV.U6.3 (In+)
- net DIV.U1.XTAL1: now reaches DIV.XTAL1.1
- net DIV.U1.XTAL1: now also DIV.C1.1
- net DIV.U1.XTAL2: now reaches DIV.XTAL1.2
- net DIV.U1.XTAL2: now also DIV.C2.1
- net ARef: now reaches DIV.U3.6 (OUT)
- net ARef: now also DIV.U1.32 (AREF)
- net OC1A: now reaches DIV.JP3.2 (B)
- net OC1A: now also DIV.U1.19 (PD5)
- net at DIV.R2.1: now also DIV.JP1.2 (B), DIV.PL2.1 (Pin_1), DIV.PL2.2 (Pin_2)
- net PD1: now reaches DIV.R2.2
- net PD1: now also DIV.U1.15 (PD1)
- net INT0: now reaches DIV.LED1.1 (K)
- net INT0: now also DIV.PL5.3 (Pin_3), DIV.U1.16 (PD2)
- net at DIV.LED1.2 (A): now also DIV.R1.1
- net TTL/Switch: now reaches DIV.PL6.2 (Pin_2)
- net ADC0: now reaches DIV.PL5.1 (Pin_1)
- net ADC0: now also DIV.U1.40 (PA0)
- net ADC1: now reaches DIV.PL5.2 (Pin_2)
- net ADC1: now also DIV.U1.39 (PA1)
- net INT1: now reaches DIV.PL5.4 (Pin_4)
- net INT1: now also DIV.U1.17 (PD3)
- net In 10A: now reaches DIV.SW3.8 (11)
- net PB0: now reaches DIV.U1.1 (PB0)
- net DIV.U1:XTAL2: now reaches DIV.U1.12 (XTAL2)
- net DIV.U1:XTAL1: now reaches DIV.U1.13 (XTAL1)
- net PB1: now reaches DIV.U1.2 (PB1)
- net OC2: now reaches DIV.U1.21 (PD7)
- net OC2: now also DIV.JP5.2 (B)
- net INT2: now reaches DIV.U1.3 (PB2)
- net DCmidProt: now reaches DIV.U1.36 (PA4)
- net OC0: now reaches DIV.U1.4 (PB3)
- net PB4: now reaches DIV.U1.5 (PB4)
- net MOSI: now reaches DIV.U1.6 (PB5)
- net MOSI: now also DIV.PL4.1 (Pin_1)
- net MISO: now reaches DIV.U1.7 (PB6)
- net MISO: now also DIV.PL4.9 (Pin_9)
- net PB7: now reaches DIV.U1.8 (PB7)
- net PB7: now also DIV.PL4.7 (Pin_7)
- net Reset: now reaches DIV.U1.9 (~{RESET})
- net Reset: now also DIV.PL4.5 (Pin_5), DIV.R7.2
- no-connect marks 4 -> 17
Other:
- note added: "+2,50000V"
- note added: "Messbereichs-Steuerung"
- moved on the sheet: DIV.C13, DIV.C14, DIV.C16, DIV.C17, DIV.C5, DIV.C7, DIV.C9, DIV.D1, DIV.D2, DIV.D3, DIV.D4, DIV.FS1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
